File: dvi-3bit/v1.0a/dvi-3bit.sch (KiCad schematic (older format))
At the start: 32 parts, among them J1 PMOD, J2 jmp, J3 5V, J4 jmp, J5 HDMI_A_1.4, U1 VREG_3V3, U2 TFP410

Commit message: Renamed hdmi to dvi.
I am being told that using hdmi term has some legal implications so we
can't use it. *sigh*
Connections:
- no-connect marks 10 -> 11
Changed lines of the file:
@@
 EESchema Schematic File Version 4
-LIBS:hdmi-3bit-cache
+LIBS:dvi-3bit-cache
 EELAYER 26 0
 EELAYER END
@@
 encoding utf-8
 Sheet 1 1
-Title "iCEBreaker PMOD - HDMI 3bit"
+Title "iCEBreaker PMOD - 3bit DVI"
 Date ""
 Rev "V0.1a"
@@
 Wire Wire Line
 	6700 4700 6700 5000
+NoConn ~ 7650 2500
 $EndSCHEMATC

Commit message: Corrected pinout and added legend.
I made a mistake copying the pinout of the original @blackmesalabs
design. I mirroed it and now it should be correct. I also added
silkscreen legend of the pin signals.
Changed lines of the file:
@@
 L Connector_Generic:Conn_02x06_Top_Bottom J1
 U 1 1 5ADECDD2
-P 1800 4300
-F 0 "J1" H 1850 4720 50  0000 C CNN
-F 1 "PMOD" H 1850 4627 50  0000 C CNN
-F 2 "pkl_connectors:PMODHeader_2x06_P2.54mm_Horizontal" H 1800 4300 50  0001 C CNN
-F 3 "~" H 1800 4300 50  0001 C CNN
-F 4 "conn-th-01in-6-2-hdr-ra" H 1800 4300 50  0001 C CNN "Key"
-F 5 "ANY" H 1800 4300 50  0001 C CNN "Source"
-	1    1800 4300
-	1    0    0    -1
+P 1900 4300
+F 0 "J1" H 1950 4720 50  0000 C CNN
+F 1 "PMOD" H 1950 4627 50  0000 C CNN
+F 2 "pkl_connectors:PMODHeader_2x06_P2.54mm_Horizontal" H 1900 4300 50  0001 C CNN
+F 3 "~" H 1900 4300 50  0001 C CNN
+F 4 "conn-th-01in-6-2-hdr-ra" H 1900 4300 50  0001 C CNN "Key"
+F 5 "ANY" H 1900 4300 50  0001 C CNN "Source"
+	1    1900 4300
+	-1   0    0    -1
 $EndComp
 Wire Wire Line
@@
 Wire Wire Line
 	1600 4600 1500 4600
-Wire Wire Line
-	1500 4600 1500 3800
 Wire Wire Line
 	2100 4600 2200 4600
@@
 	6700 4700 6700 5000
 NoConn ~ 7650 2500
+Wire Wire Line
+	1500 4600 1500 3800
 $EndSCHEMATC
