File: 7segment/v1.0a/7segment.kicad_pcb (KiCad board)
At the start: 4 copper layers, 37 x 20.3 mm, 7 parts, among them J1 PMOD, U1 LTD-6910HR, U2 NL27WZ14

Commit message: Removed the two inner layers for the 7segment. We only need two here.
Other:
- copper layers 4 -> 2
Changed lines of the file:
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@@
   (layers
     (0 F.Cu signal)
-    (1 In1.Cu signal)
-    (2 In2.Cu signal)
     (31 B.Cu signal)
     (32 B.Adhes user)
