File: 7segment/v1.0a/7segment.kicad_pcb (KiCad board)
At the start: 2 copper layers, 37 x 20.3 mm, 7 parts, among them J1 PMOD, U1 LTD-6910HR, U2 NL27WZ14

Commit message: Some global cleanup.
Parts:
- added REF**: null_Logo_SilkS_6.5mm, pkl_logos:null_Logo_SilkS_6.5mm, B.Cu at (50.7, 40.2)
Other:
- board text added: "NULL"
Changed lines of the file:
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@@
-(kicad_pcb (version 20171130) (host pcbnew 5.0.2-bee76a0~70~ubuntu18.04.1)
+(kicad_pcb (version 20171130) (host pcbnew 5.1.5-52549c5~86~ubuntu19.10.1)
   (general
     (thickness 1.6)
-    (drawings 62)
+    (drawings 63)
     (tracks 111)
     (zones 0)
-    (modules 7)
+    (modules 8)
     (nets 23)
   )
@@
     (zone_45_only no)
     (trace_min 0.15)
-    (segment_width 0.2)
-    (edge_width 0.15)
     (via_size 0.5)
     (via_drill 0.3)
@@
     (uvia_min_size 0.2)
     (uvia_min_drill 0.1)
+    (edge_width 0.15)
+    (segment_width 0.2)
     (pcb_text_width 0.3)
     (pcb_text_size 1.5 1.5)
@@
     (add_net "Net-(U1-Pad4)")
     (add_net "Net-(U1-Pad9)")
+  )
+  (module pkl_logos:null_Logo_SilkS_6.5mm (layer B.Cu)
+    (at 50.7 40.2 90)
+    (fp_text reference REF** (at 0 -4.55 90) (layer B.Fab) hide
+      (effects (font (size 1 1) (thickness 0.15)) (justify mirror))
+    )
+    (fp_text value null_Logo_SilkS_6.5mm (at 0 4.55 90) (layer B.Fab) hide
+      (effects (font (size 1 1) (thickness 0.15)) (justify mirror))
+    )
+    (fp_arc (start -0.4 -0.2) (end -0.7 -0.2) (angle 180) (layer B.SilkS) (width 0.15))
+    (fp_line (start 1 -0.5) (end 1.5 -0.5) (layer B.SilkS) (width 0.15))
+    (fp_line (start 1 0.5) (end 1 -0.5) (layer B.SilkS) (width 0.15))
+    (fp_line (start 0.2 -0.5) (end 0.7 -0.5) (layer B.SilkS) (width 0.15))
+    (fp_line (start 0.2 0.5) (end 0.2 -0.5) (layer B.SilkS) (width 0.15))
+    (fp_line (start -0.1 -0.2) (end -0.1 0.5) (layer B.SilkS) (width 0.15))
+    (fp_line (start -0.7 0.5) (end -0.7 -0.2) (layer B.SilkS) (width 0.15))
+    (fp_line (start -1 -0.5) (end -1 0.5) (layer B.SilkS) (width 0.15))
+    (fp_line (start -1.5 0.5) (end -1 -0.5) (layer B.SilkS) (width 0.15))
+    (fp_line (start -1.5 -0.5) (end -1.5 0.5) (layer B.SilkS) (width 0.15))
+    (fp_line (start 3.25 3.25) (end -3.25 3.25) (layer B.SilkS) (width 0.26))
+    (fp_line (start -3.25 3.25) (end -3.25 -3.25) (layer B.SilkS) (width 0.26))
+    (fp_line (start 3.25 3.25) (end 3.25 -3.25) (layer B.SilkS) (width 0.26))
+    (fp_line (start -3.25 -3.25) (end 3.25 -3.25) (layer B.SilkS) (width 0.26))
   )
   (module pkl_dipol:C_0402 (layer B.Cu)
@@
     )
   )
+  (gr_text NULL (at 46.5 40.2 270) (layer B.SilkS)
+    (effects (font (size 1 1) (thickness 0.25)) (justify mirror))
+  )
   (gr_text CC-BY-SA (at 30.798 40.2 270) (layer B.SilkS)
