File: 7segment/v1.0a/7segment.sch (KiCad schematic (older format))
At the start: 7 parts, among them J1 PMOD, U1 LTD-6910HR, U2 NL27WZ14

Commit message: Added bom tracking keys.
Parts:
- R1, R2: Key (none) -> res-0402cv-array-4-330
- U1: Key (none) -> led-disp-ltd-6910hr
- U2: Key (none) -> ic-sot363-dual-inverter-nl27wz14
Changed lines of the file:
@@
 L pkl_misc:NL27WZ14 U2
 U 1 1 5BBFC7DD
-P 7700 4800
-F 0 "U2" H 7700 5170 50  0000 C CNN
-F 1 "NL27WZ14" H 7700 5077 50  0000 C CNN
-F 2 "Package_TO_SOT_SMD:SOT-363_SC-70-6" H 7720 4800 50  0001 C CNN
-F 3 "" H 7720 4800 50  0001 C CNN
-	1    7700 4800
-	1    0    0    -1
-$EndComp
-Wire Wire Line
-	7300 4800 7100 4800
-Wire Wire Line
-	7100 4800 7100 5100
-Wire Wire Line
-	8100 4800 8300 4800
-Wire Wire Line
-	8300 4800 8300 4500
+P 7000 4500
+F 0 "U2" H 7000 4870 50  0000 C CNN
+F 1 "NL27WZ14" H 7000 4777 50  0000 C CNN
+F 2 "Package_TO_SOT_SMD:SOT-363_SC-70-6" H 7020 4500 50  0001 C CNN
+F 3 "" H 7020 4500 50  0001 C CNN
+F 4 "ic-sot363-dual-inverter-nl27wz14" H 0   0   50  0001 C CNN "Key"
+	1    7000 4500
+	1    0    0    -1
+$EndComp
+Wire Wire Line
+	6600 4500 6400 4500
+Wire Wire Line
+	6400 4500 6400 4800
+Wire Wire Line
+	7400 4500 7600 4500
+Wire Wire Line
+	7600 4500 7600 4200
 $Comp
 L power:GND #PWR08
 U 1 1 5BBFC7E8
-P 7100 5100
-F 0 "#PWR08" H 7100 4850 50  0001 C CNN
-F 1 "GND" H 7105 4924 50  0000 C CNN
-F 2 "" H 7100 5100 50  0001 C CNN
-F 3 "" H 7100 5100 50  0001 C CNN
-	1    7100 5100
+P 6400 4800
+F 0 "#PWR08" H 6400 4550 50  0001 C CNN
+F 1 "GND" H 6405 4624 50  0000 C CNN
+F 2 "" H 6400 4800 50  0001 C CNN
+F 3 "" H 6400 4800 50  0001 C CNN
+	1    6400 4800
 	1    0    0    -1
 $EndComp
@@
 L power:+3V3 #PWR09
 U 1 1 5BBFC7EE
-P 8300 4500
-F 0 "#PWR09" H 8300 4350 50  0001 C CNN
-F 1 "+3V3" H 8315 4676 50  0000 C CNN
-F 2 "" H 8300 4500 50  0001 C CNN
-F 3 "" H 8300 4500 50  0001 C CNN
-	1    8300 4500
-	1    0    0    -1
-$EndComp
-Wire Wire Line
-	7300 4700 7000 4700
-Wire Wire Line
-	8100 4700 8200 4700
-Wire Wire Line
-	8200 4700 8200 5100
-Wire Wire Line
-	8200 5100 7200 5100
-Wire Wire Line
-	7200 5100 7200 4900
-Wire Wire Line
-	7200 4900 7300 4900
-Wire Wire Line
-	8100 4900 8400 4900
+P 7600 4200
+F 0 "#PWR09" H 7600 4050 50  0001 C CNN
+F 1 "+3V3" H 7615 4376 50  0000 C CNN
+F 2 "" H 7600 4200 50  0001 C CNN
+F 3 "" H 7600 4200 50  0001 C CNN
+	1    7600 4200
+	1    0    0    -1
+$EndComp
+Wire Wire Line
+	6600 4400 6300 4400
+Wire Wire Line
+	7400 4400 7500 4400
+Wire Wire Line
+	7500 4400 7500 4800
+Wire Wire Line
+	7500 4800 6500 4800
+Wire Wire Line
+	6500 4800 6500 4600
+Wire Wire Line
+	6500 4600 6600 4600
+Wire Wire Line
+	7400 4600 7700 4600
 Text Label 4500 3500 0    50   ~ 0
 AA
@@
 Text Label 3600 3800 2    50   ~ 0
 CAT
-Text Label 7000 4700 2    50   ~ 0
+Text Label 6300 4400 2    50   ~ 0
 CATx
 Wire Wire Line
-	8200 4700 8400 4700
-Connection ~ 8200 4700
-Text Label 8400 4700 0    50   ~ 0
+	7500 4400 7700 4400
+Connection ~ 7500 4400
+Text Label 7700 4400 0    50   ~ 0
 CAT1
-Text Label 8400 4900 0    50   ~ 0
+Text Label 7700 4600 0    50   ~ 0
 CAT2
 $Comp
 L pkl_misc:LTD-6910HR U1
 U 1 1 5BC026F5
-P 7600 3200
-F 0 "U1" H 7600 3870 50  0000 C CNN
-F 1 "LTD-6910HR" H 7600 3777 50  0000 C CNN
-F 2 "pkl_led:LTD-6910HR" H 8000 2500 50  0001 C CNN
-F 3 "" H 8000 2500 50  0001 C CNN
-	1    7600 3200
+P 7000 3350
+F 0 "U1" H 7000 4020 50  0000 C CNN
+F 1 "LTD-6910HR" H 7000 3927 50  0000 C CNN
+F 2 "pkl_led:LTD-6910HR" H 7400 2650 50  0001 C CNN
+F 3 "" H 7400 2650 50  0001 C CNN
+F 4 "led-disp-ltd-6910hr" H 0   0   50  0001 C CNN "Key"
+	1    7000 3350
 	1    0    0    -1
 $EndComp
@@
 F 2 "pkl_dipol:R_Array_Convex_4x0402" H 4900 3500 60  0001 C CNN
 F 3 "" H 4900 3500 60  0000 C CNN
+F 4 "res-0402cv-array-4-330" H 0   0   50  0001 C CNN "Key"
 	1    4900 3500
 	0    1    1    0
 $EndComp
 Wire Wire Line
-	6900 2900 6800 2900
-Wire Wire Line
-	6900 2800 6800 2800
-Wire Wire Line
-	8300 2800 8400 2800
-Wire Wire Line
-	6900 3000 6800 3000
-Wire Wire Line
-	6900 3100 6800 3100
-Wire Wire Line
-	6900 3200 6800 3200
-Wire Wire Line
-	6900 3300 6800 3300
-Wire Wire Line
-	6900 3400 6800 3400
-Wire Wire Line
-	6900 3500 6800 3500
-Wire Wire Line
-	8300 2900 8400 2900
-Wire Wire Line
-	8300 3000 8400 3000
-Wire Wire Line
-	8300 3100 8400 3100
-Wire Wire Line
-	8300 3200 8400 3200
-Wire Wire Line
-	8300 3300 8400 3300
-Wire Wire Line
-	8300 3400 8400 3400
-Wire Wire Line
-	8300 3500 8400 3500
-NoConn ~ 8300 3600
-NoConn ~ 6900 3600
-Text Label 6800 2800 2    50   ~ 0
+	6300 3050 6200 3050
+Wire Wire Line
+	6300 2950 6200 2950
+Wire Wire Line
+	7700 2950 7800 2950
+Wire Wire Line
+	6300 3150 6200 3150
+Wire Wire Line
+	6300 3250 6200 3250
+Wire Wire Line
+	6300 3350 6200 3350
+Wire Wire Line
+	6300 3450 6200 3450
+Wire Wire Line
+	6300 3550 6200 3550
+Wire Wire Line
+	6300 3650 6200 3650
+Wire Wire Line
+	7700 3050 7800 3050
+Wire Wire Line
+	7700 3150 7800 3150
+Wire Wire Line
+	7700 3250 7800 3250
+Wire Wire Line
+	7700 3350 7800 3350
+Wire Wire Line
+	7700 3450 7800 3450
+Wire Wire Line
+	7700 3550 7800 3550
+Wire Wire Line
+	7700 3650 7800 3650
+NoConn ~ 7700 3750
+NoConn ~ 6300 3750
+Text Label 6200 2950 2    50   ~ 0
 CAT1
-Text Label 8400 2800 0    50   ~ 0
+Text Label 7800 2950 0    50   ~ 0
 CAT2
-Text Label 6800 2900 2    50   ~ 0
+Text Label 6200 3050 2    50   ~ 0
 AAx
-Text Label 6800 3000 2    50   ~ 0
+Text Label 6200 3150 2    50   ~ 0
 ABx
-Text Label 6800 3100 2    50   ~ 0
+Text Label 6200 3250 2    50   ~ 0
 ACx
-Text Label 6800 3200 2    50   ~ 0
+Text Label 6200 3350 2    50   ~ 0
 ADx
-Text Label 6800 3300 2    50   ~ 0
+Text Label 6200 3450 2    50   ~ 0
 AEx
-Text Label 6800 3400 2    50   ~ 0
+Text Label 6200 3550 2    50   ~ 0
 AFx
-Text Label 6800 3500 2    50   ~ 0
+Text Label 6200 3650 2    50   ~ 0
 AGx
-Text Label 8400 2900 0    50   ~ 0
+Text Label 7800 3050 0    50   ~ 0
 AAx
-Text Label 8400 3000 0    50   ~ 0
+Text Label 7800 3150 0    50   ~ 0
 ABx
-Text Label 8400 3100 0    50   ~ 0
+Text Label 7800 3250 0    50   ~ 0
 ACx
-Text Label 8400 3200 0    50   ~ 0
+Text Label 7800 3350 0    50   ~ 0
 ADx
-Text Label 8400 3300 0    50   ~ 0
+Text Label 7800 3450 0    50   ~ 0
 AEx
-Text Label 8400 3400 0    50   ~ 0
+Text Label 7800 3550 0    50   ~ 0
 AFx
-Text Label 8400 3500 0    50   ~ 0
+Text Label 7800 3650 0    50   ~ 0
 AGx
 $Comp
@@
 F 2 "pkl_dipol:R_Array_Convex_4x0402" H 3200 3500 60  0001 C CNN
 F 3 "" H 3200 3500 60  0000 C CNN
+F 4 "res-0402cv-array-4-330" H 3200 3500 50  0001 C CNN "Key"
 	2    3200 3500
 	0    -1   1    0
@@
 F 2 "pkl_dipol:R_Array_Convex_4x0402" H 4900 3600 60  0001 C CNN
 F 3 "" H 4900 3600 60  0000 C CNN
+F 4 "res-0402cv-array-4-330" H 0   0   50  0001 C CNN "Key"
 	3    4900 3600
 	0    1    1    0
@@
 F 2 "pkl_dipol:R_Array_Convex_4x0402" H 3200 3600 60  0001 C CNN
 F 3 "" H 3200 3600 60  0000 C CNN
+F 4 "res-0402cv-array-4-330" H 0   0   50  0001 C CNN "Key"
 	4    3200 3600
 	0    -1   1    0
@@
 F 2 "pkl_dipol:R_Array_Convex_4x0402" H 4900 3700 60  0001 C CNN
 F 3 "" H 4900 3700 60  0000 C CNN
+F 4 "res-0402cv-array-4-330" H 4900 3700 50  0001 C CNN "Key"
 	1    4900 3700
 	0    1    1    0
@@
 F 2 "pkl_dipol:R_Array_Convex_4x0402" H 3200 3700 60  0001 C CNN
 F 3 "" H 3200 3700 60  0000 C CNN
+F 4 "res-0402cv-array-4-330" H 0   0   50  0001 C CNN "Key"
 	2    3200 3700
 	0    -1   1    0
@@
 F 2 "pkl_dipol:R_Array_Convex_4x0402" H 4900 3800 60  0001 C CNN
 F 3 "" H 4900 3800 60  0000 C CNN
+F 4 "res-0402cv-array-4-330" H 0   0   50  0001 C CNN "Key"
 	3    4900 3800
 	0    1    1    0
@@
 F 2 "pkl_dipol:R_Array_Convex_4x0402" H 3200 3800 60  0001 C CNN
 F 3 "" H 3200 3800 60  0000 C CNN
+F 4 "res-0402cv-array-4-330" H 0   0   50  0001 C CNN "Key"
 	4    3200 3800
 	0    -1   1    0
