File: led-panel/v1.0a/led-panel.kicad_pcb (KiCad board)
At the start: 2 copper layers, 34.6 x 40 mm, 13 parts, among them J1 5V, J2 PMOD, J3 jmp, J4 PMOD, J5 jmp, J6 Conn_02x08_Odd_Even, U1 SN74LVC8T245, U2 SN74LVC8T245

Commit message: Corrected signal names for the LED panel PMOD.
The BLANK, LATCH, SCLK are all positive logic not negative.
Connections:
- net /i~BLANK renamed /iBLANK
- net /i~LATCH renamed /iLATCH
- net /i~SCLK renamed /iSCLK
- net /~BLANK renamed /BLANK
- net /~LATCH renamed /LATCH
- net /~SCLK renamed /SCLK
