File: led-panel/v1.2a/led-panel.sch (KiCad schematic (older format))
At the start: 25 parts, among them J1 5V, J2 PMOD, J3 jmp, J4 PMOD, J5 jmp, J6 Conn_02x08_Odd_Even, J7 jmp, U1 SN74LVC8T245, U2 SN74LVC8T245

Commit message: Corrected led panel pmod project name.
Parts:
- J1: Key conn-th-01in-6-2-hdr-ra -> conn-th-01in-2-1-rec
- J2, J4: Key (none) -> conn-th-01in-6-2-hdr-ra
- J6: Key (none) -> conn-th-01in-8-2-hdr
- R5, R6, R7, R8: Key (none) -> res-0402cv-array-4-33
Changed lines of the file:
@@
 encoding utf-8
 Sheet 1 1
-Title "iCEBreaker PMOD - Hyperram"
+Title "iCEBreaker PMOD - LED Panel HUB75E"
 Date ""
 Rev "V1.2a"
@@
 F 2 "pkl_connectors:PMODHeader_2x06_P2.54mm_Horizontal" H 4700 2500 50  0001 C CNN
 F 3 "~" H 4700 2500 50  0001 C CNN
-F 4 "ANY" H 4700 2500 50  0001 C CNN "Source"
+F 4 "conn-th-01in-6-2-hdr-ra" H 4700 2500 50  0001 C CNN "Key"
+F 5 "ANY" H 4700 2500 50  0001 C CNN "Source"
 	1    4700 2500
 	-1   0    0    -1
@@
 F 2 "Connector_PinHeader_2.54mm:PinHeader_2x08_P2.54mm_Vertical" H 9300 3200 50  0001 C CNN
 F 3 "~" H 9300 3200 50  0001 C CNN
+F 4 "conn-th-01in-8-2-hdr" H 9300 3200 50  0001 C CNN "Key"
 	1    9300 3200
 	1    0    0    -1
@@
 F 2 "Connector_PinHeader_2.54mm:PinHeader_2x01_P2.54mm_Vertical" H 4600 3550 50  0001 C CNN
 F 3 "~" H 4600 3550 50  0001 C CNN
-F 4 "conn-th-01in-6-2-hdr-ra" H 4600 3550 50  0001 C CNN "Key"
+F 4 "conn-th-01in-2-1-rec" H 4600 3550 50  0001 C CNN "Key"
 F 5 "ANY" H 4600 3550 50  0001 C CNN "Source"
 	1    4600 3550
@@
 F 2 "pkl_connectors:PMODHeader_2x06_P2.54mm_Horizontal" H 4700 4600 50  0001 C CNN
 F 3 "~" H 4700 4600 50  0001 C CNN
-F 4 "ANY" H 4700 4600 50  0001 C CNN "Source"
+F 4 "conn-th-01in-6-2-hdr-ra" H 4700 4600 50  0001 C CNN "Key"
+F 5 "ANY" H 4700 4600 50  0001 C CNN "Source"
 	1    4700 4600
 	-1   0    0    -1
@@
 F 2 "pkl_dipol:R_Array_Convex_4x0402" H 7800 2200 60  0001 C CNN
 F 3 "" H 7800 2200 60  0000 C CNN
+F 4 "res-0402cv-array-4-33" H 0   0   50  0001 C CNN "Key"
 	1    7800 2200
 	0    -1   1    0
@@
 F 2 "pkl_dipol:R_Array_Convex_4x0402" H 7800 2300 60  0001 C CNN
 F 3 "" H 7800 2300 60  0000 C CNN
+F 4 "res-0402cv-array-4-33" H 0   0   50  0001 C CNN "Key"
 	2    7800 2300
 	0    -1   1    0
@@
 F 2 "pkl_dipol:R_Array_Convex_4x0402" H 7800 2400 60  0001 C CNN
 F 3 "" H 7800 2400 60  0000 C CNN
+F 4 "res-0402cv-array-4-33" H 0   0   50  0001 C CNN "Key"
 	3    7800 2400
 	0    -1   -1   0
@@
 F 2 "pkl_dipol:R_Array_Convex_4x0402" H 7800 2500 60  0001 C CNN
 F 3 "" H 7800 2500 60  0000 C CNN
+F 4 "res-0402cv-array-4-33" H 0   0   50  0001 C CNN "Key"
 	4    7800 2500
 	0    -1   1    0
@@
 F 2 "pkl_dipol:R_Array_Convex_4x0402" H 7800 2600 60  0001 C CNN
 F 3 "" H 7800 2600 60  0000 C CNN
+F 4 "res-0402cv-array-4-33" H 0   0   50  0001 C CNN "Key"
 	1    7800 2600
 	0    -1   1    0
@@
 F 2 "pkl_dipol:R_Array_Convex_4x0402" H 7800 2700 60  0001 C CNN
 F 3 "" H 7800 2700 60  0000 C CNN
+F 4 "res-0402cv-array-4-33" H 0   0   50  0001 C CNN "Key"
 	2    7800 2700
 	0    -1   1    0
@@
 F 2 "pkl_dipol:R_Array_Convex_4x0402" H 7800 2800 60  0001 C CNN
 F 3 "" H 7800 2800 60  0000 C CNN
+F 4 "res-0402cv-array-4-33" H 0   0   50  0001 C CNN "Key"
 	3    7800 2800
 	0    -1   1    0
@@
 F 2 "pkl_dipol:R_Array_Convex_4x0402" H 7800 2900 60  0001 C CNN
 F 3 "" H 7800 2900 60  0000 C CNN
+F 4 "res-0402cv-array-4-33" H 0   0   50  0001 C CNN "Key"
 	4    7800 2900
 	0    -1   1    0
@@
 F 2 "pkl_dipol:R_Array_Convex_4x0402" H 7800 4300 60  0001 C CNN
 F 3 "" H 7800 4300 60  0000 C CNN
+F 4 "res-0402cv-array-4-33" H 0   0   50  0001 C CNN "Key"
 	1    7800 4300
 	0    -1   1    0
@@
 F 2 "pkl_dipol:R_Array_Convex_4x0402" H 7800 4400 60  0001 C CNN
 F 3 "" H 7800 4400 60  0000 C CNN
+F 4 "res-0402cv-array-4-33" H 0   0   50  0001 C CNN "Key"
 	2    7800 4400
 	0    -1   1    0
@@
 F 2 "pkl_dipol:R_Array_Convex_4x0402" H 7800 4500 60  0001 C CNN
 F 3 "" H 7800 4500 60  0000 C CNN
+F 4 "res-0402cv-array-4-33" H 0   0   50  0001 C CNN "Key"
 	3    7800 4500
 	0    -1   1    0
@@
 F 2 "pkl_dipol:R_Array_Convex_4x0402" H 7800 4600 60  0001 C CNN
 F 3 "" H 7800 4600 60  0000 C CNN
+F 4 "res-0402cv-array-4-33" H 0   0   50  0001 C CNN "Key"
 	4    7800 4600
 	0    -1   1    0
@@
 F 2 "pkl_dipol:R_Array_Convex_4x0402" H 7800 4700 60  0001 C CNN
 F 3 "" H 7800 4700 60  0000 C CNN
+F 4 "res-0402cv-array-4-33" H 0   0   50  0001 C CNN "Key"
 	1    7800 4700
 	0    -1   1    0
@@
 F 2 "pkl_dipol:R_Array_Convex_4x0402" H 7800 4800 60  0001 C CNN
 F 3 "" H 7800 4800 60  0000 C CNN
+F 4 "res-0402cv-array-4-33" H 0   0   50  0001 C CNN "Key"
 	2    7800 4800
 	0    -1   1    0
@@
 F 2 "pkl_dipol:R_Array_Convex_4x0402" H 7800 4900 60  0001 C CNN
 F 3 "" H 7800 4900 60  0000 C CNN
+F 4 "res-0402cv-array-4-33" H 0   0   50  0001 C CNN "Key"
 	3    7800 4900
 	0    -1   1    0
@@
 F 2 "pkl_dipol:R_Array_Convex_4x0402" H 7800 5000 60  0001 C CNN
 F 3 "" H 7800 5000 60  0000 C CNN
+F 4 "res-0402cv-array-4-33" H 0   0   50  0001 C CNN "Key"
 	4    7800 5000
 	0    -1   1    0
