File: led-panel/v1.2a/led-panel.kicad_pcb (KiCad board)
At the start: 2 copper layers, 35 x 40 mm, 25 parts, among them J1 5V, J2 PMOD, J3 jmp, J4 PMOD, J5 jmp, J6 Conn_02x08_Odd_Even, J7 jmp, U1 SN74LVC8T245, U2 SN74LVC8T245

Commit message: Corrected led panel pmod project name.
Other:
- rule solder_mask_min_width: 0.25 -> 0.05
Changed lines of the file:
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@@
-(kicad_pcb (version 20171130) (host pcbnew 5.0.1-33cea8e~68~ubuntu18.04.1)
+(kicad_pcb (version 20171130) (host pcbnew 5.0.2-bee76a0~70~ubuntu18.04.1)
   (general
     (thickness 0.8)
@@
   (page A4)
   (title_block
-    (title "iCEBreaker PMOD - Hyperram")
+    (title "iCEBreaker PMOD - LED Panel HUB75E")
     (rev V1.2a)
     (company 1BitSquared)
@@
     (pad_drill 0)
     (pad_to_mask_clearance 0.05)
-    (solder_mask_min_width 0.25)
+    (solder_mask_min_width 0.05)
     (aux_axis_origin 0 0)
     (grid_origin 37.4 44)

Commit message: Some global cleanup.
Parts:
- added REF**: null_Logo_SilkS_5mm, pkl_logos:null_Logo_SilkS_5mm, B.Cu at (57.4, 44.2)
Other:
- board text added: "NULL"
Changed lines of the file:
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@@
-(kicad_pcb (version 20171130) (host pcbnew 5.0.2-bee76a0~70~ubuntu18.04.1)
+(kicad_pcb (version 20171130) (host pcbnew 5.1.5-52549c5~86~ubuntu19.10.1)
   (general
     (thickness 0.8)
-    (drawings 151)
+    (drawings 152)
     (tracks 266)
     (zones 0)
-    (modules 25)
+    (modules 26)
     (nets 59)
   )
@@
     (zone_45_only yes)
     (trace_min 0.2)
-    (segment_width 0.15)
-    (edge_width 0.15)
     (via_size 0.5)
     (via_drill 0.3)
@@
     (uvia_min_size 0.2)
     (uvia_min_drill 0.1)
+    (edge_width 0.15)
+    (segment_width 0.15)
     (pcb_text_width 0.3)
     (pcb_text_size 1.5 1.5)
@@
     (add_net "Net-(R4-Pad1)")
   )
+  (module pkl_logos:null_Logo_SilkS_5mm locked (layer B.Cu)
+    (at 57.4 44.2 90)
+    (fp_text reference REF** (at 0 -4 90) (layer B.Fab) hide
+      (effects (font (size 1 1) (thickness 0.15)) (justify mirror))
+    )
+    (fp_text value null_Logo_SilkS_5mm (at 0 4 90) (layer B.Fab) hide
+      (effects (font (size 1 1) (thickness 0.15)) (justify mirror))
+    )
+    (fp_arc (start -0.4 -0.2) (end -0.7 -0.2) (angle 180) (layer B.SilkS) (width 0.15))
+    (fp_line (start 1 -0.5) (end 1.5 -0.5) (layer B.SilkS) (width 0.15))
+    (fp_line (start 1 0.5) (end 1 -0.5) (layer B.SilkS) (width 0.15))
+    (fp_line (start 0.2 -0.5) (end 0.7 -0.5) (layer B.SilkS) (width 0.15))
+    (fp_line (start 0.2 0.5) (end 0.2 -0.5) (layer B.SilkS) (width 0.15))
+    (fp_line (start -0.1 0.5) (end -0.1 -0.2) (layer B.SilkS) (width 0.15))
+    (fp_line (start -0.7 0.5) (end -0.7 -0.2) (layer B.SilkS) (width 0.15))
+    (fp_line (start -1 -0.5) (end -1 0.5) (layer B.SilkS) (width 0.15))
+    (fp_line (start -1.5 0.5) (end -1 -0.5) (layer B.SilkS) (width 0.15))
+    (fp_line (start -1.5 -0.5) (end -1.5 0.5) (layer B.SilkS) (width 0.15))
+    (fp_line (start 2.5 2.5) (end -2.5 2.5) (layer B.SilkS) (width 0.2))
+    (fp_line (start -2.5 2.5) (end -2.5 -2.5) (layer B.SilkS) (width 0.2))
+    (fp_line (start 2.5 2.5) (end 2.5 -2.5) (layer B.SilkS) (width 0.2))
+    (fp_line (start -2.5 -2.5) (end 2.5 -2.5) (layer B.SilkS) (width 0.2))
+  )
   (module pkl_dipol:C_0402 (layer F.Cu)
     (at 49.8 35.4 90)
@@
     )
   )
+  (gr_text NULL (at 54 44 270) (layer B.SilkS)
+    (effects (font (size 0.75 0.75) (thickness 0.1875)) (justify mirror))
+  )
   (gr_text GND (at 38.8 45.5 270) (layer B.SilkS)
