File: dvi-24bit/v1.0a/dvi-24bit.sch (KiCad schematic (older format))
At the start: 38 parts, among them J1 PMOD, J10 sj, J2 PMOD, J3 jmp, J4 5V, J5 3v3_5v_sel, J6 HDMI_A_1.4, J7 sj, J8 sj, J9 sj, U1 VREG_3V3, U2 SII164

Commit message: Moved CLK, set default DK.
* Moved CLK: This is for the iCEBreaker. It allows the use of a separate
clock and ability to rotate the clock wave by 90deg.
* As we have DKEN on by default, we should also set the jumpers to a
sane default. In this case we use the internal default of the part that
is 0b100.

Thanks for the suggestions @smunaut.
Parts:
- J7, J8, J9: footprint pkl_jumpers:J_0903 -> pkl_jumpers:J_NCNO_0903_15; symbol pkl_misc:pkl_double_jumper -> pkl_misc:pkl_double_jumper_ncno
Connections:
- net +3V3: now also J8.3, J9.3; no longer J8.1, J9.1
- net CLK: now also J1.3 (Pin_3); no longer J1.2 (Pin_2)
- net D0: now also J1.8 (Pin_8); no longer J1.3 (Pin_3)
- net D1: now also J1.2 (Pin_2); no longer J1.8 (Pin_8)
- net GND: now also J8.1, J9.1; no longer J8.3, J9.3
Changed lines of the file:
@@
 Text Label 2300 6000 0    50   ~ 0
 HS
-Text Label 2300 5800 0    50   ~ 0
+Text Label 2300 5900 0    50   ~ 0
 CLK
 $Comp
@@
 Wire Wire Line
 	2100 4200 2300 4200
-Text Label 2300 5900 0    50   ~ 0
+Text Label 1400 5800 2    50   ~ 0
 D0
 Text Label 2300 5700 0    50   ~ 0
 D3
-Text Label 1400 5800 2    50   ~ 0
+Text Label 2300 5800 0    50   ~ 0
 D1
 Text Label 1400 5700 2    50   ~ 0
@@
 	7800 3800 7800 4300
 $Comp
-L pkl_misc:pkl_double_jumper J8
+L pkl_misc:pkl_double_jumper_ncno J8
 U 1 1 5D36E9CC
 P 4000 6000
 F 0 "J8" H 3900 6050 50  0000 R CNN
 F 1 "sj" H 4200 6050 50  0000 R CNN
-F 2 "pkl_jumpers:J_0903" H 3950 6000 50  0001 C CNN
+F 2 "pkl_jumpers:J_NCNO_0903_15" H 3950 6000 50  0001 C CNN
 F 3 "" H 3950 6000 50  0001 C CNN
 	1    4000 6000
-	0    1    1    0
-$EndComp
-$Comp
-L pkl_misc:pkl_double_jumper J7
+	0    1    -1   0
+$EndComp
+$Comp
+L pkl_misc:pkl_double_jumper_ncno J7
 U 1 1 5D3730B1
 P 3800 6000
 F 0 "J7" H 3700 6050 50  0000 R CNN
 F 1 "sj" H 4000 6050 50  0000 R CNN
-F 2 "pkl_jumpers:J_0903" H 3750 6000 50  0001 C CNN
+F 2 "pkl_jumpers:J_NCNO_0903_15" H 3750 6000 50  0001 C CNN
 F 3 "" H 3750 6000 50  0001 C CNN
 	1    3800 6000
@@
 $EndComp
 $Comp
-L pkl_misc:pkl_double_jumper J9
+L pkl_misc:pkl_double_jumper_ncno J9
 U 1 1 5D44E723
 P 4200 6000
 F 0 "J9" H 4100 6050 50  0000 R CNN
 F 1 "sj" H 4400 6050 50  0000 R CNN
-F 2 "pkl_jumpers:J_0903" H 4150 6000 50  0001 C CNN
+F 2 "pkl_jumpers:J_NCNO_0903_15" H 4150 6000 50  0001 C CNN
 F 3 "" H 4150 6000 50  0001 C CNN
 	1    4200 6000
-	0    1    1    0
-$EndComp
-$Comp
+	0    1    -1   0
+$EndComp
+$Comp
