File: 7segment/v1.1a/7segment.kicad_pcb (KiCad board)
At the start: 2 copper layers, 41 x 20.3 mm, 7 parts, among them J1 PMOD, U1 SN450561N, U2 NL27WZ14

Commit message: Some global cleanup.
Parts:
- added REF**: null_Logo_SilkS_6.5mm, pkl_logos:null_Logo_SilkS_6.5mm, B.Cu at (52.7, 40.2)
Other:
- board text added: "NULL"
