File: 7segment/v1.1a/7segment.sch (KiCad schematic (older format))
At the start: 7 parts, among them J1 PMOD, U1 SN450561N, U2 NL27WZ14

Commit message: Some global cleanup.
Other:
- note added: "Dual Inverter"
- note added: "Pmod Connector"
Changed lines of the file:
@@
 	0    -1   1    0
 $EndComp
+Text Notes 6550 5050 0    100  ~ 0
+Dual Inverter
+Text Notes 3450 2800 0    100  ~ 0
+Pmod Connector
 $EndSCHEMATC
