File: dip-switch/v1.0a/dip-switch.kicad_pcb (KiCad board)
At the start: 2 copper layers, 37 x 16 mm, 4 parts, among them J1 PMOD, SW1 SW_DIP_x08

Commit message: Some global cleanup.
Parts:
- added REF**: null_Logo_SilkS_5mm, pkl_logos:null_Logo_SilkS_5mm, B.Cu at (54.4, 40.2)
Other:
- board text added: "NULL"
Changed lines of the file:
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@@
-(kicad_pcb (version 20171130) (host pcbnew 5.0.2-bee76a0~70~ubuntu18.04.1)
+(kicad_pcb (version 20171130) (host pcbnew 5.1.5-52549c5~86~ubuntu19.10.1)
   (general
     (thickness 1.6)
-    (drawings 24)
+    (drawings 25)
     (tracks 81)
     (zones 0)
-    (modules 4)
+    (modules 5)
     (nets 11)
   )
@@
     (zone_45_only no)
     (trace_min 0.2)
-    (segment_width 0.2)
-    (edge_width 0.15)
     (via_size 0.5)
     (via_drill 0.3)
@@
     (uvia_min_size 0.2)
     (uvia_min_drill 0.1)
+    (edge_width 0.15)
+    (segment_width 0.2)
     (pcb_text_width 0.3)
     (pcb_text_size 1.5 1.5)
@@
     (add_net /DIP8)
     (add_net GND)
+  )
+  (module pkl_logos:null_Logo_SilkS_5mm locked (layer B.Cu)
+    (at 54.42 40.2 90)
+    (fp_text reference REF** (at 0 -4 90) (layer B.Fab)
+      (effects (font (size 1 1) (thickness 0.15)) (justify mirror))
+    )
+    (fp_text value null_Logo_SilkS_5mm (at 0 4 90) (layer B.Fab)
+      (effects (font (size 1 1) (thickness 0.15)) (justify mirror))
+    )
+    (fp_arc (start -0.4 -0.2) (end -0.7 -0.2) (angle 180) (layer B.SilkS) (width 0.15))
+    (fp_line (start 1 -0.5) (end 1.5 -0.5) (layer B.SilkS) (width 0.15))
+    (fp_line (start 1 0.5) (end 1 -0.5) (layer B.SilkS) (width 0.15))
+    (fp_line (start 0.2 -0.5) (end 0.7 -0.5) (layer B.SilkS) (width 0.15))
+    (fp_line (start 0.2 0.5) (end 0.2 -0.5) (layer B.SilkS) (width 0.15))
+    (fp_line (start -0.1 0.5) (end -0.1 -0.2) (layer B.SilkS) (width 0.15))
+    (fp_line (start -0.7 0.5) (end -0.7 -0.2) (layer B.SilkS) (width 0.15))
+    (fp_line (start -1 -0.5) (end -1 0.5) (layer B.SilkS) (width 0.15))
+    (fp_line (start -1.5 0.5) (end -1 -0.5) (layer B.SilkS) (width 0.15))
+    (fp_line (start -1.5 -0.5) (end -1.5 0.5) (layer B.SilkS) (width 0.15))
+    (fp_line (start 2.5 2.5) (end -2.5 2.5) (layer B.SilkS) (width 0.2))
+    (fp_line (start -2.5 2.5) (end -2.5 -2.5) (layer B.SilkS) (width 0.2))
+    (fp_line (start 2.5 2.5) (end 2.5 -2.5) (layer B.SilkS) (width 0.2))
+    (fp_line (start -2.5 -2.5) (end 2.5 -2.5) (layer B.SilkS) (width 0.2))
   )
   (module Button_Switch_THT:SW_DIP_SPSTx08_Slide_9.78x22.5mm_W7.62mm_P2.54mm (layer F.Cu)
@@
     )
   )
+  (gr_text NULL (at 50.61 40.2 270) (layer B.SilkS)
+    (effects (font (size 0.75 0.75) (thickness 0.1875)) (justify mirror))
+  )
   (gr_text ON (at 42.8 38.2 90) (layer F.SilkS)
