File: dip-switch/v1.1a/dip-switch.kicad_pcb (KiCad board)
At the start: 2 copper layers, 38 x 16 mm, 4 parts, among them J1 PMOD, SW1 SW_DIP_x08

Commit message: Some global cleanup.
Parts:
- added REF**: null_Logo_SilkS_5mm, pkl_logos:null_Logo_SilkS_5mm, B.Cu at (55.5, 40.2)
Other:
- board text added: "NULL"
