File: dvi-12bit/v1.0b/dvi-12bit.kicad_pcb (KiCad board)
At the start: 4 copper layers, 40 x 40.8 mm, 33 parts, among them J1 PMOD, J2 PMOD, J3 jmp, J4 5V, J5 3v3_5v_sel, J6 HDMI_A_1.4, U1 VREG_3V3, U2 TFP410

Commit message: Some global cleanup.
Parts:
- added REF**: null_Logo_SilkS_10mm, pkl_logos:null_Logo_SilkS_10mm, B.Cu at (51.6, 40.2)
Other:
- board text added: "NULL"
Changed lines of the file:
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@@
-(kicad_pcb (version 20171130) (host pcbnew 5.0.2-bee76a0~70~ubuntu18.04.1)
+(kicad_pcb (version 20171130) (host pcbnew 5.1.5-52549c5~86~ubuntu19.10.1)
   (general
     (thickness 1.6)
-    (drawings 99)
+    (drawings 100)
     (tracks 306)
     (zones 0)
-    (modules 33)
+    (modules 34)
     (nets 52)
   )
@@
     (zone_45_only no)
     (trace_min 0.15)
-    (segment_width 0.2)
-    (edge_width 0.15)
     (via_size 0.5)
     (via_drill 0.3)
@@
     (uvia_min_size 0.2)
     (uvia_min_drill 0.1)
+    (edge_width 0.15)
+    (segment_width 0.2)
     (pcb_text_width 0.3)
     (pcb_text_size 1.5 1.5)
@@
     (pad_to_mask_clearance 0.05)
     (solder_mask_min_width 0.25)
-    (aux_axis_origin 0 0)
-    (grid_origin 30 40.2)
+    (aux_axis_origin 70 60.6)
     (visible_elements FFFFFF1F)
     (pcbplotparams
@@
       (drillshape 0)
       (scaleselection 1)
-      (outputdirectory "gerber"))
+      (outputdirectory ""))
   )
   (net 0 "")
@@
     (add_net "Net-(U2-Pad8)")
   )
+  (module pkl_logos:null_Logo_SilkS_10mm (layer B.Cu)
+    (at 51.6 40.2 90)
+    (fp_text reference REF** (at 0 -6 90) (layer B.Fab) hide
+      (effects (font (size 1 1) (thickness 0.15)) (justify mirror))
+    )
+    (fp_text value null_Logo_SilkS_10mm (at 0 6.35 90) (layer B.Fab) hide
+      (effects (font (size 1 1) (thickness 0.15)) (justify mirror))
+    )
+    (fp_arc (start -0.4 -0.2) (end -0.7 -0.2) (angle 180) (layer B.SilkS) (width 0.15))
+    (fp_line (start 1 -0.5) (end 1.5 -0.5) (layer B.SilkS) (width 0.15))
+    (fp_line (start 1 0.5) (end 1 -0.5) (layer B.SilkS) (width 0.15))
+    (fp_line (start 0.2 -0.5) (end 0.7 -0.5) (layer B.SilkS) (width 0.15))
+    (fp_line (start 0.2 0.5) (end 0.2 -0.5) (layer B.SilkS) (width 0.15))
+    (fp_line (start -0.1 0.5) (end -0.1 -0.2) (layer B.SilkS) (width 0.15))
+    (fp_line (start -0.7 0.5) (end -0.7 -0.2) (layer B.SilkS) (width 0.15))
+    (fp_line (start -1 -0.5) (end -1 0.5) (layer B.SilkS) (width 0.15))
+    (fp_line (start -1.5 0.5) (end -1 -0.5) (layer B.SilkS) (width 0.15))
+    (fp_line (start -1.5 -0.5) (end -1.5 0.5) (layer B.SilkS) (width 0.15))
+    (fp_line (start 5 5) (end -5 5) (layer B.SilkS) (width 0.4))
+    (fp_line (start -5 5) (end -5 -5) (layer B.SilkS) (width 0.4))
+    (fp_line (start 5 5) (end 5 -5) (layer B.SilkS) (width 0.4))
+    (fp_line (start -5 -5) (end 5 -5) (layer B.SilkS) (width 0.4))
+  )
   (module pkl_jumpers:J_NCNO_0903_30 (layer B.Cu)
     (at 60.1 46.6 270)
@@
     )
   )
+  (gr_text NULL (at 44.7 40.1 270) (layer B.SilkS)
+    (effects (font (size 1.5 1.5) (thickness 0.3)) (justify mirror))
+  )
   (gr_text +5V (at 38.9 40.2 270) (layer B.SilkS)
