File: dvi-12bit/v1.1a/dvi-12bit.kicad_pcb (KiCad board)
At the start: 4 copper layers, 40 x 40.8 mm, 39 parts, among them J1 PMOD, J10 sj, J2 PMOD, J3 jmp, J4 5V, J5 3v3_5v_sel, J6 HDMI_A_1.4, J7 sj, J8 sj, J9 sj, U1 VREG_3V3, U2 SII164

Commit message: Some global cleanup.
Parts:
- REF**: value 1b2_Logo_SilkS_7.5mm -> null_Logo_SilkS_7.5mm; footprint pkl_logos:1b2_Logo_SilkS_7.5mm -> pkl_logos:null_Logo_SilkS_7.5mm
Other:
- board text added: "NULL"
- board text removed: "1BitSquared"
Changed lines of the file:
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@@
-(kicad_pcb (version 20171130) (host pcbnew 5.1.2-f72e74a~84~ubuntu18.04.1)
+(kicad_pcb (version 20171130) (host pcbnew 5.1.5-52549c5~86~ubuntu19.10.1)
   (general
     (thickness 1.6)
-    (drawings 104)
+    (drawings 106)
     (tracks 349)
     (zones 0)
@@
     (add_net "Net-(J1-Pad12)")
     (add_net "Net-(J5-Pad2)")
-    (add_net "Net-(J6-Pad13)")
-    (add_net "Net-(J6-Pad14)")
-    (add_net "Net-(J6-Pad15)")
-    (add_net "Net-(J6-Pad16)")
-    (add_net "Net-(J6-Pad19)")
-    (add_net "Net-(U2-Pad11)")
-  )
-  (module pkl_logos:1b2_Logo_SilkS_7.5mm (layer B.Cu)
+  )
+  (module pkl_logos:null_Logo_SilkS_7.5mm (layer B.Cu)
     (at 47.6 37.5 90)
     (fp_text reference REF** (at 0 -5 90) (layer B.Fab)
       (effects (font (size 1 1) (thickness 0.15)) (justify mirror))
     )
-    (fp_text value 1b2_Logo_SilkS_7.5mm (at 0 5 90) (layer B.Fab)
+    (fp_text value null_Logo_SilkS_7.5mm (at 0 5 90) (layer B.Fab)
       (effects (font (size 1 1) (thickness 0.15)) (justify mirror))
     )
-    (fp_line (start -0.75 0.75) (end -0.75 3.75) (layer B.SilkS) (width 0.3))
-    (fp_line (start -0.75 3.75) (end -3.75 3.75) (layer B.SilkS) (width 0.3))
-    (fp_line (start -3.75 3.75) (end -3.75 0.75) (layer B.SilkS) (width 0.3))
-    (fp_line (start -3.75 0.75) (end -0.75 0.75) (layer B.SilkS) (width 0.3))
-    (fp_line (start -0.75 3.75) (end 0 3) (layer B.SilkS) (width 0.3))
-    (fp_line (start 0 3) (end 0 0) (layer B.SilkS) (width 0.3))
-    (fp_line (start 0 0) (end -0.75 0.75) (layer B.SilkS) (width 0.3))
-    (fp_line (start -3.75 0.75) (end -3 0) (layer B.SilkS) (width 0.3))
-    (fp_line (start -3 0) (end 0 0) (layer B.SilkS) (width 0.3))
-    (fp_line (start 3 3) (end 0.75 3) (layer B.SilkS) (width 0.3))
-    (fp_line (start 0.75 3) (end 0.75 -0.75) (layer B.SilkS) (width 0.3))
-    (fp_line (start 0.75 -0.75) (end -3 -0.75) (layer B.SilkS) (width 0.3))
-    (fp_line (start -3 -0.75) (end -3 -3) (layer B.SilkS) (width 0.3))
-    (fp_line (start -3 -3) (end 3 -3) (layer B.SilkS) (width 0.3))
-    (fp_line (start 3 -3) (end 3 3) (layer B.SilkS) (width 0.3))
-    (fp_line (start 3 3) (end 3.75 2.25) (layer B.SilkS) (width 0.3))
-    (fp_line (start 3.75 2.25) (end 3.75 -3.75) (layer B.SilkS) (width 0.3))
-    (fp_line (start 3.75 -3.75) (end 3 -3) (layer B.SilkS) (width 0.3))
-    (fp_line (start -3 -3) (end -2.25 -3.75) (layer B.SilkS) (width 0.3))
-    (fp_line (start -2.25 -3.75) (end 3.75 -3.75) (layer B.SilkS) (width 0.3))
+    (fp_line (start 1 -0.5) (end 1.5 -0.5) (layer B.SilkS) (width 0.15))
+    (fp_line (start 1 0.5) (end 1 -0.5) (layer B.SilkS) (width 0.15))
+    (fp_line (start 0.2 -0.5) (end 0.7 -0.5) (layer B.SilkS) (width 0.15))
+    (fp_line (start 0.2 0.5) (end 0.2 -0.5) (layer B.SilkS) (width 0.15))
+    (fp_line (start -0.1 -0.2) (end -0.1 0.5) (layer B.SilkS) (width 0.15))
+    (fp_arc (start -0.4 -0.2) (end -0.7 -0.2) (angle 180) (layer B.SilkS) (width 0.15))
+    (fp_line (start -0.7 0.5) (end -0.7 -0.2) (layer B.SilkS) (width 0.15))
+    (fp_line (start -1 -0.5) (end -1 0.5) (layer B.SilkS) (width 0.15))
+    (fp_line (start -1.5 0.5) (end -1 -0.5) (layer B.SilkS) (width 0.15))
+    (fp_line (start -1.5 -0.5) (end -1.5 0.5) (layer B.SilkS) (width 0.15))
+    (fp_line (start 3.75 3.75) (end -3.75 3.75) (layer B.SilkS) (width 0.3))
+    (fp_line (start -3.75 3.75) (end -3.75 -3.75) (layer B.SilkS) (width 0.3))
+    (fp_line (start 3.75 3.75) (end 3.75 -3.75) (layer B.SilkS) (width 0.3))
+    (fp_line (start -3.75 -3.75) (end 3.75 -3.75) (layer B.SilkS) (width 0.3))
   )
   (module pkl_jumpers:J_0903 (layer B.Cu)
@@
     )
   )
+  (gr_line (start 61.2 47.7) (end 71.02 32.7) (layer Dwgs.User) (width 0.15))
+  (gr_line (start 71.02 47.7) (end 61.2 32.7) (layer Dwgs.User) (width 0.15))
   (gr_text DK3 (at 49.7 46.9 270) (layer B.SilkS)
     (effects (font (size 1 1) (thickness 0.2)) (justify mirror))
@@
     (effects (font (size 1 1) (thickness 0.2)) (justify mirror))
   )
-  (gr_text 1BitSquared (at 42.3 37.15 270) (layer B.SilkS)
+  (gr_text NULL (at 42.3 37.15 270) (layer B.SilkS)
     (effects (font (size 1.5 1.5) (thickness 0.3)) (justify mirror))
   )
@@
   (segment (start 39 50.6) (end 39 44.3) (width 0.15) (layer F.Cu) (net 5))
   (segment (start 39 44.3) (end 41.1 42.2) (width 0.15) (layer F.Cu) (net 5))
-  (segment (start 46.75 46.95) (end 46.8 46.9) (width 0.15) (layer F.Cu) (net 40))
-  (segment (start 45.5 46.95) (end 46.75 46.95) (width 0.15) (layer F.Cu) (net 40))
-  (segment (start 46.85 46.95) (end 46.8 46.9) (width 0.15) (layer F.Cu) (net 40))
-  (segment (start 48.1 46.95) (end 46.85 46.95) (width 0.15) (layer F.Cu) (net 40))
-  (segment (start 46.75 46.85) (end 46.8 46.9) (width 0.15) (layer F.Cu) (net 40))
-  (segment (start 46.75 46.1) (end 46.75 46.85) (width 0.15) (layer F.Cu) (net 40))
-  (via (at 46.75 46.1) (size 0.5) (drill 0.3) (layers F.Cu B.Cu) (net 40))
-  (segment (start 46.75 44.8) (end 46.75 46.1) (width 0.15) (layer F.Cu) (net 40))
-  (segment (start 54.25 33.4) (end 54.25 31.95) (width 0.15) (layer F.Cu) (net 40))
-  (via (at 54.6 34.6) (size 0.5) (drill 0.3) (layers F.Cu B.Cu) (net 40))
-  (segment (start 54.25 34.25) (end 54.6 34.6) (width 0.15) (layer F.Cu) (net 40))
-  (segment (start 54.25 33.4) (end 54.25 34.25) (width 0.15) (layer F.Cu) (net 40))
-  (segment (start 54 35.2) (end 54.6 34.6) (width 0.3) (layer In1.Cu) (net 40))
-  (segment (start 46.550001 35.649999) (end 47 35.2) (width 0.3) (layer In1.Cu) (net 40))
-  (segment (start 47 35.2) (end 54 35.2) (width 0.3) (layer In1.Cu) (net 40))
-  (segment (start 46.550001 45.950001) (end 46.550001 35.649999) (width 0.3) (layer In1.Cu) (net 40))
-  (segment (start 46.75 46.1) (end 46.7 46.1) (width 0.3) (layer In1.Cu) (net 40))
-  (segment (start 46.7 46.1) (end 46.550001 45.950001) (width 0.3) (layer In1.Cu) (net 40))
   (segment (start 49.1 46.95) (end 50.1 46.95) (width 0.15) (layer F.Cu) (net 6))
   (segment (start 49 46.95) (end 49.1 46.95) (width 0.15) (layer F.Cu) (net 6))
@@
   (segment (start 53.75 44.8) (end 53.75 45.55) (width 0.15) (layer F.Cu) (net 13))
   (segment (start 53.75 45.55) (end 54.37498 46.17498) (width 0.15) (layer F.Cu) (net 13))
-  (segment (start 57.7 44.15) (end 57.65 44.1) (width 0.15) (layer F.Cu) (net 41))
-  (segment (start 57.7 45.4) (end 57.7 44.15) (width 0.15) (layer F.Cu) (net 41))
-  (segment (start 57.7 44.05) (end 57.65 44.1) (width 0.15) (layer F.Cu) (net 41))
-  (segment (start 57.7 42.8) (end 57.7 44.05) (width 0.15) (layer F.Cu) (net 41))
-  (segment (start 57.25 42.35) (end 57.7 42.8) (width 0.15) (layer F.Cu) (net 41))
-  (segment (start 56.2 42.35) (end 57.25 42.35) (width 0.15) (layer F.Cu) (net 41))
   (segment (start 59.996998 40.95) (end 60.5 40.95) (width 0.15) (layer F.Cu) (net 14))
   (segment (start 59.897008 40.85001) (end 59.996998 40.95) (width 0.15) (layer F.Cu) (net 14))
@@
   (segment (start 36.6 22.42) (end 36.62 22.42) (width 0.15) (layer F.Cu) (net 39))
   (segment (start 45.3 30.3) (end 50.55 30.3) (width 0.15) (layer F.Cu) (net 39))
+  (segment (start 46.75 46.95) (end 46.8 46.9) (width 0.15) (layer F.Cu) (net 40))
+  (segment (start 45.5 46.95) (end 46.75 46.95) (width 0.15) (layer F.Cu) (net 40))
+  (segment (start 46.85 46.95) (end 46.8 46.9) (width 0.15) (layer F.Cu) (net 40))
+  (segment (start 48.1 46.95) (end 46.85 46.95) (width 0.15) (layer F.Cu) (net 40))
+  (segment (start 46.75 46.85) (end 46.8 46.9) (width 0.15) (layer F.Cu) (net 40))
+  (segment (start 46.75 46.1) (end 46.75 46.85) (width 0.15) (layer F.Cu) (net 40))
+  (via (at 46.75 46.1) (size 0.5) (drill 0.3) (layers F.Cu B.Cu) (net 40))
+  (segment (start 46.75 44.8) (end 46.75 46.1) (width 0.15) (layer F.Cu) (net 40))
+  (segment (start 54.25 33.4) (end 54.25 31.95) (width 0.15) (layer F.Cu) (net 40))
+  (via (at 54.6 34.6) (size 0.5) (drill 0.3) (layers F.Cu B.Cu) (net 40))
+  (segment (start 54.25 34.25) (end 54.6 34.6) (width 0.15) (layer F.Cu) (net 40))
+  (segment (start 54.25 33.4) (end 54.25 34.25) (width 0.15) (layer F.Cu) (net 40))
+  (segment (start 54 35.2) (end 54.6 34.6) (width 0.3) (layer In1.Cu) (net 40))
+  (segment (start 46.550001 35.649999) (end 47 35.2) (width 0.3) (layer In1.Cu) (net 40))
+  (segment (start 47 35.2) (end 54 35.2) (width 0.3) (layer In1.Cu) (net 40))
+  (segment (start 46.550001 45.950001) (end 46.550001 35.649999) (width 0.3) (layer In1.Cu) (net 40))
+  (segment (start 46.75 46.1) (end 46.7 46.1) (width 0.3) (layer In1.Cu) (net 40))
+  (segment (start 46.7 46.1) (end 46.550001 45.950001) (width 0.3) (layer In1.Cu) (net 40))
   (segment (start 53.1 46.95) (end 52.864105 46.714105) (width 0.15) (layer F.Cu) (net 40))
   (segment (start 47.25 46.6) (end 52.5 46.6) (width 0.3) (layer In1.Cu) (net 40))
@@
   (via (at 52.864105 46.235895) (size 0.5) (drill 0.3) (layers F.Cu B.Cu) (net 40))
   (segment (start 52.5 46.6) (end 52.864105 46.235895) (width 0.3) (layer In1.Cu) (net 40))
+  (segment (start 57.7 44.15) (end 57.65 44.1) (width 0.15) (layer F.Cu) (net 41))
+  (segment (start 57.7 45.4) (end 57.7 44.15) (width 0.15) (layer F.Cu) (net 41))
+  (segment (start 57.7 44.05) (end 57.65 44.1) (width 0.15) (layer F.Cu) (net 41))
+  (segment (start 57.7 42.8) (end 57.7 44.05) (width 0.15) (layer F.Cu) (net 41))
+  (segment (start 57.25 42.35) (end 57.7 42.8) (width 0.15) (layer F.Cu) (net 41))
+  (segment (start 56.2 42.35) (end 57.25 42.35) (width 0.15) (layer F.Cu) (net 41))
   (segment (start 44.8 34.3) (end 44.8 35.35) (width 0.15) (layer F.Cu) (net 41))
   (via (at 57.7 46.3) (size 0.5) (drill 0.3) (layers F.Cu B.Cu) (net 41))
