File: dvi-4bit/v1.0a/dvi-4bit.kicad_pcb (KiCad board)
At the start: 4 copper layers, 37 x 20.3 mm, 32 parts, among them J1 PMOD, J2 jmp, J3 5V, J4 3v3_5v_sel, J5 HDMI_A_1.4, U1 VREG_3V3, U2 TFP410

Commit message: Some global cleanup.
Parts:
- added REF**: null_Logo_SilkS_10mm, pkl_logos:null_Logo_SilkS_10mm, B.Cu at (48.6, 40.2)
Other:
- rule solder_mask_min_width: 0.25 -> 0.05
- board text added: "NULL"
