File: hyperram/v1.0a/ibp-hyperram.kicad_pcb (KiCad board)
At the start: 2 copper layers, 20.5 x 42 mm, 6 parts, among them J2 PMOD, J4 PMOD, U1 S70KL1281

Commit message: Some global cleanup.
Parts:
- added REF**: null_Logo_SilkS_6.5mm, pkl_logos:null_Logo_SilkS_6.5mm, B.Cu at (52.3, 44.0)
Other:
- board text added: "NULL"
Changed lines of the file:
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@@
-(kicad_pcb (version 20171130) (host pcbnew 5.0.0-fee4fd1~66~ubuntu18.04.1)
+(kicad_pcb (version 20171130) (host pcbnew 5.1.5-52549c5~86~ubuntu19.10.1)
   (general
     (thickness 0.8)
-    (drawings 54)
+    (drawings 55)
     (tracks 102)
     (zones 0)
-    (modules 6)
+    (modules 7)
     (nets 24)
   )
@@
     (zone_45_only yes)
     (trace_min 0.2)
-    (segment_width 0.15)
-    (edge_width 0.15)
     (via_size 0.5)
     (via_drill 0.3)
@@
     (uvia_min_size 0.2)
     (uvia_min_drill 0.1)
+    (edge_width 0.15)
+    (segment_width 0.15)
     (pcb_text_width 0.3)
     (pcb_text_size 1.5 1.5)
@@
     (add_net "Net-(U1-PadC2)")
     (add_net "Net-(U1-PadC5)")
+  )
+  (module pkl_logos:null_Logo_SilkS_6.5mm (layer B.Cu)
+    (at 52.3 44 90)
+    (fp_text reference REF** (at 0 -4.55 90) (layer B.Fab)
+      (effects (font (size 1 1) (thickness 0.15)) (justify mirror))
+    )
+    (fp_text value null_Logo_SilkS_6.5mm (at 0 4.55 90) (layer B.Fab)
+      (effects (font (size 1 1) (thickness 0.15)) (justify mirror))
+    )
+    (fp_arc (start -0.4 -0.2) (end -0.7 -0.2) (angle 180) (layer B.SilkS) (width 0.15))
+    (fp_line (start 1 -0.5) (end 1.5 -0.5) (layer B.SilkS) (width 0.15))
+    (fp_line (start 1 0.5) (end 1 -0.5) (layer B.SilkS) (width 0.15))
+    (fp_line (start 0.2 -0.5) (end 0.7 -0.5) (layer B.SilkS) (width 0.15))
+    (fp_line (start 0.2 0.5) (end 0.2 -0.5) (layer B.SilkS) (width 0.15))
+    (fp_line (start -0.1 -0.2) (end -0.1 0.5) (layer B.SilkS) (width 0.15))
+    (fp_line (start -0.7 0.5) (end -0.7 -0.2) (layer B.SilkS) (width 0.15))
+    (fp_line (start -1 -0.5) (end -1 0.5) (layer B.SilkS) (width 0.15))
+    (fp_line (start -1.5 0.5) (end -1 -0.5) (layer B.SilkS) (width 0.15))
+    (fp_line (start -1.5 -0.5) (end -1.5 0.5) (layer B.SilkS) (width 0.15))
+    (fp_line (start 3.25 3.25) (end -3.25 3.25) (layer B.SilkS) (width 0.26))
+    (fp_line (start -3.25 3.25) (end -3.25 -3.25) (layer B.SilkS) (width 0.26))
+    (fp_line (start 3.25 3.25) (end 3.25 -3.25) (layer B.SilkS) (width 0.26))
+    (fp_line (start -3.25 -3.25) (end 3.25 -3.25) (layer B.SilkS) (width 0.26))
   )
   (module pkl_dipol:C_0402 (layer F.Cu)
@@
     )
   )
+  (gr_text NULL (at 47.6 44 270) (layer B.SilkS)
+    (effects (font (size 1.25 1.25) (thickness 0.3)) (justify mirror))
+  )
   (gr_text "V1.0a\n(C) 2018\n1BitSquared" (at 57.4 62.5) (layer B.SilkS)
