File: hyperram/v1.0b/ibp-hyperram.kicad_pcb (KiCad board)
At the start: 2 copper layers, 20.5 x 42 mm, 6 parts, among them J2 PMOD, J4 PMOD, U1 S70KL1281

Commit message: Some global cleanup.
Parts:
- added REF**: null_Logo_SilkS_7.5mm, pkl_logos:null_Logo_SilkS_7.5mm, B.Cu at (52.8, 44.0)
Other:
- board text added: "NULL"
Changed lines of the file:
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@@
-(kicad_pcb (version 20171130) (host pcbnew 5.0.0-fee4fd1~66~ubuntu18.04.1)
+(kicad_pcb (version 20171130) (host pcbnew 5.1.5-52549c5~86~ubuntu19.10.1)
   (general
     (thickness 0.8)
-    (drawings 54)
+    (drawings 55)
     (tracks 105)
     (zones 0)
-    (modules 6)
+    (modules 7)
     (nets 24)
   )
@@
     (zone_45_only yes)
     (trace_min 0.2)
-    (segment_width 0.15)
-    (edge_width 0.15)
     (via_size 0.5)
     (via_drill 0.3)
@@
     (uvia_min_size 0.2)
     (uvia_min_drill 0.1)
+    (edge_width 0.15)
+    (segment_width 0.15)
     (pcb_text_width 0.3)
     (pcb_text_size 1.5 1.5)
@@
     (pad_drill 0)
     (pad_to_mask_clearance 0.05)
+    (solder_mask_min_width 0.25)
     (aux_axis_origin 0 0)
     (grid_origin 44 44)
@@
     (add_net "Net-(U1-PadC2)")
     (add_net "Net-(U1-PadC5)")
+  )
+  (module pkl_logos:null_Logo_SilkS_7.5mm (layer B.Cu)
+    (at 52.8 44 90)
+    (fp_text reference REF** (at 0 -5 90) (layer B.Fab)
+      (effects (font (size 1 1) (thickness 0.15)) (justify mirror))
+    )
+    (fp_text value null_Logo_SilkS_7.5mm (at 0 5 90) (layer B.Fab)
+      (effects (font (size 1 1) (thickness 0.15)) (justify mirror))
+    )
+    (fp_line (start 1 -0.5) (end 1.5 -0.5) (layer B.SilkS) (width 0.15))
+    (fp_line (start 1 0.5) (end 1 -0.5) (layer B.SilkS) (width 0.15))
+    (fp_line (start 0.2 -0.5) (end 0.7 -0.5) (layer B.SilkS) (width 0.15))
+    (fp_line (start 0.2 0.5) (end 0.2 -0.5) (layer B.SilkS) (width 0.15))
+    (fp_line (start -0.1 -0.2) (end -0.1 0.5) (layer B.SilkS) (width 0.15))
+    (fp_arc (start -0.4 -0.2) (end -0.7 -0.2) (angle 180) (layer B.SilkS) (width 0.15))
+    (fp_line (start -0.7 0.5) (end -0.7 -0.2) (layer B.SilkS) (width 0.15))
+    (fp_line (start -1 -0.5) (end -1 0.5) (layer B.SilkS) (width 0.15))
+    (fp_line (start -1.5 0.5) (end -1 -0.5) (layer B.SilkS) (width 0.15))
+    (fp_line (start -1.5 -0.5) (end -1.5 0.5) (layer B.SilkS) (width 0.15))
+    (fp_line (start 3.75 3.75) (end -3.75 3.75) (layer B.SilkS) (width 0.3))
+    (fp_line (start -3.75 3.75) (end -3.75 -3.75) (layer B.SilkS) (width 0.3))
+    (fp_line (start 3.75 3.75) (end 3.75 -3.75) (layer B.SilkS) (width 0.3))
+    (fp_line (start -3.75 -3.75) (end 3.75 -3.75) (layer B.SilkS) (width 0.3))
   )
   (module pkl_dipol:C_0402 (layer F.Cu)
@@
     )
   )
+  (gr_text NULL (at 47.5 44 270) (layer B.SilkS)
+    (effects (font (size 1.25 1.25) (thickness 0.3)) (justify mirror))
+  )
   (gr_text "V1.0b\n(C) 2018\n1BitSquared" (at 57.4 62.5) (layer B.SilkS)
     (effects (font (size 0.75 0.75) (thickness 0.1875)) (justify left mirror))
@@
   (via (at 48.7 42.8) (size 0.5) (drill 0.3) (layers F.Cu B.Cu) (net 10))
   (segment (start 48.7 44) (end 48.7 42.8) (width 0.2) (layer B.Cu) (net 10))
-  (segment (start 48.7 38) (end 48.7 42.8) (width 0.2) (layer F.Cu) (net 10))
+  (segment (start 48.7 38) (end 48.7 42.8) (width 0.25) (layer F.Cu) (net 10))
   (segment (start 45.8 35.1) (end 48.7 38) (width 0.2) (layer F.Cu) (net 10))
   (segment (start 41.46 33.84) (end 42.72 35.1) (width 0.2) (layer F.Cu) (net 10))
