File: led-panel-single-mini/v1.0a/led-panel-single-mini.kicad_pcb (KiCad board)
At the start: 2 copper layers, 37 x 20 mm, 22 parts, among them J1 5V, J2 jmp, J3 Conn_02x08_Odd_Even, J4 PMOD, J5 jmp, U1 SN74LVC8T245, U2 NL27WZ14, U3 74HC4024, U4 74VHC574

Commit message: Some global cleanup.
Parts:
- added REF**: null_Logo_SilkS_5mm, pkl_logos:null_Logo_SilkS_5mm, B.Cu at (60.5, 41.2)
Other:
- board text added: "NULL"
Changed lines of the file:
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@@
-(kicad_pcb (version 20171130) (host pcbnew 5.0.2-bee76a0~70~ubuntu18.04.1)
+(kicad_pcb (version 20171130) (host pcbnew 5.1.5-52549c5~86~ubuntu19.10.1)
   (general
     (thickness 0.8)
-    (drawings 94)
+    (drawings 95)
     (tracks 290)
     (zones 0)
-    (modules 22)
+    (modules 23)
     (nets 67)
   )
@@
     (zone_45_only yes)
     (trace_min 0.2)
-    (segment_width 0.15)
-    (edge_width 0.15)
     (via_size 0.5)
     (via_drill 0.3)
@@
     (uvia_min_size 0.2)
     (uvia_min_drill 0.1)
+    (edge_width 0.15)
+    (segment_width 0.15)
     (pcb_text_width 0.3)
     (pcb_text_size 1.5 1.5)
@@
     (pad_to_mask_clearance 0.05)
     (solder_mask_min_width 0.05)
-    (aux_axis_origin 0 0)
+    (aux_axis_origin 37.4 54)
     (grid_origin 37.4 44)
     (visible_elements FFFFFF1F)
@@
       (viasonmask false)
       (mode 1)
-      (useauxorigin false)
+      (useauxorigin true)
       (hpglpennumber 1)
       (hpglpenspeed 20)
@@
     (add_net "Net-(U4-Pad9)")
   )
+  (module pkl_logos:null_Logo_SilkS_5mm locked (layer B.Cu)
+    (at 60.49361 41.194674)
+    (fp_text reference REF** (at 0 -4) (layer B.Fab) hide
+      (effects (font (size 1 1) (thickness 0.15)) (justify mirror))
+    )
+    (fp_text value null_Logo_SilkS_5mm (at 0 4) (layer B.Fab) hide
+      (effects (font (size 1 1) (thickness 0.15)) (justify mirror))
+    )
+    (fp_arc (start -0.4 -0.2) (end -0.7 -0.2) (angle 180) (layer B.SilkS) (width 0.15))
+    (fp_line (start 1 -0.5) (end 1.5 -0.5) (layer B.SilkS) (width 0.15))
+    (fp_line (start 1 0.5) (end 1 -0.5) (layer B.SilkS) (width 0.15))
+    (fp_line (start 0.2 -0.5) (end 0.7 -0.5) (layer B.SilkS) (width 0.15))
+    (fp_line (start 0.2 0.5) (end 0.2 -0.5) (layer B.SilkS) (width 0.15))
+    (fp_line (start -0.1 0.5) (end -0.1 -0.2) (layer B.SilkS) (width 0.15))
+    (fp_line (start -0.7 0.5) (end -0.7 -0.2) (layer B.SilkS) (width 0.15))
+    (fp_line (start -1 -0.5) (end -1 0.5) (layer B.SilkS) (width 0.15))
+    (fp_line (start -1.5 0.5) (end -1 -0.5) (layer B.SilkS) (width 0.15))
+    (fp_line (start -1.5 -0.5) (end -1.5 0.5) (layer B.SilkS) (width 0.15))
+    (fp_line (start 2.5 2.5) (end -2.5 2.5) (layer B.SilkS) (width 0.2))
+    (fp_line (start -2.5 2.5) (end -2.5 -2.5) (layer B.SilkS) (width 0.2))
+    (fp_line (start 2.5 2.5) (end 2.5 -2.5) (layer B.SilkS) (width 0.2))
+    (fp_line (start -2.5 -2.5) (end 2.5 -2.5) (layer B.SilkS) (width 0.2))
+  )
   (module Connector_PinHeader_1.27mm:PinHeader_2x08_P1.27mm_Vertical (layer F.Cu)
     (at 69.785 39.555)
@@
     )
   )
+  (gr_text NULL (at 60.69361 37.794674 180) (layer B.SilkS)
+    (effects (font (size 0.75 0.75) (thickness 0.1875)) (justify mirror))
+  )
   (gr_text "HUB75E LED Panel Driver PMOD\nV1.0a Mini" (at 52 35.9) (layer F.SilkS)
