File: quadhyperram/v1.0a/ibp-quadhyperram.kicad_pcb (KiCad board)
At the start: 4 copper layers, 20.5 x 42 mm, 23 parts, among them J1 PMOD, J2 PMOD, J3 vcc_sel, U1 S70KL1281, U2 S70KL1281, U3 S70KL1281, U4 S70KL1281, U5 VREG_1V8

Commit message: Added power selection jumper legend.
Other:
- board text added: "1V8"
- board text added: "VCC"
Changed lines of the file:
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@@
   (general
     (thickness 0.8)
-    (drawings 34)
+    (drawings 37)
     (tracks 693)
     (zones 0)
@@
     )
   )
+  (gr_text VCC (at 44.7 44.3 90) (layer B.SilkS)
+    (effects (font (size 1 1) (thickness 0.25)) (justify mirror))
+  )
+  (gr_text 3V3 (at 43.3 46.9) (layer B.SilkS)
+    (effects (font (size 1 1) (thickness 0.25)) (justify mirror))
+  )
+  (gr_text 1V8 (at 43.3 41.8) (layer B.SilkS)
+    (effects (font (size 1 1) (thickness 0.25)) (justify mirror))
+  )
   (gr_text "V1.0a\n(C) 2020\n1BitSquared" (at 57.1 62.7) (layer B.SilkS)

Commit message: Changed soldermask opening size to 0.01mm
Other:
- rule pad_to_mask_clearance: 0.05 -> 0.01
Changed lines of the file:
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@@
     (pad_size 0.5 0.6)
     (pad_drill 0)
-    (pad_to_mask_clearance 0.05)
+    (pad_to_mask_clearance 0.01)
     (aux_axis_origin 0 0)
     (grid_origin 44 44)
-    (visible_elements FFFFEF1F)
+    (visible_elements FFFFEF7F)
     (pcbplotparams
       (layerselection 0x010fc_ffffffff)

Commit message: Some global cleanup.
Parts:
- added REF**: null_Logo_SilkS_6.5mm, pkl_logos:null_Logo_SilkS_6.5mm, B.Cu at (53.7, 44.3)
Other:
- board text added: "NULL"
