File: gamepad-n-audio/gna-snes-pod/gna-snes-pod.kicad_pcb (KiCad board)
At the start: 2 copper layers, 78 x 43 mm, 12 parts, among them J1 SNES, J2 SNES, J3 Gamepads, J4 SNES, J5 SNES

Commit message: GPNA SNES: Bumped version fixed mask params.
Other:
- rule pad_to_mask_clearance: 0.05 -> 0
- board text added: "iCEBreaker SNES Gamepad Pod V1.1a 1Bitsquared 2020 CC-BY-SA"
- board text removed: "iCEBreaker SNES Gamepad Pod V1.0b 1Bitsquared 2020 CC-BY-SA"
Changed lines of the file:
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@@
     (pad_size 0.5 0.6)
     (pad_drill 0)
-    (pad_to_mask_clearance 0.05)
-    (solder_mask_min_width 0.05)
+    (pad_to_mask_clearance 0)
     (aux_axis_origin 37.4 95)
     (grid_origin 37.4 74)
@@
     (add_net VCC)
   )
+  (module pkl_logos:null_Logo_SilkS_6.5mm locked (layer F.Cu)
+    (at 43.4 89.5)
+    (attr virtual)
+    (fp_text reference REF** (at 0 4) (layer F.Fab) hide
+      (effects (font (size 1 1) (thickness 0.15)))
+    )
+    (fp_text value null_Logo_SilkS_6.5mm (at 0 -4) (layer F.Fab) hide
+      (effects (font (size 1 1) (thickness 0.15)))
+    )
+    (fp_arc (start -0.4 0.2) (end -0.7 0.2) (angle -180) (layer F.SilkS) (width 0.15))
+    (fp_line (start 1 0.5) (end 1.5 0.5) (layer F.SilkS) (width 0.15))
+    (fp_line (start 1 -0.5) (end 1 0.5) (layer F.SilkS) (width 0.15))
+    (fp_line (start 0.2 0.5) (end 0.7 0.5) (layer F.SilkS) (width 0.15))
+    (fp_line (start 0.2 -0.5) (end 0.2 0.5) (layer F.SilkS) (width 0.15))
+    (fp_line (start -0.1 0.2) (end -0.1 -0.5) (layer F.SilkS) (width 0.15))
+    (fp_line (start -0.7 -0.5) (end -0.7 0.2) (layer F.SilkS) (width 0.15))
+    (fp_line (start -1 0.5) (end -1 -0.5) (layer F.SilkS) (width 0.15))
+    (fp_line (start -1.5 -0.5) (end -1 0.5) (layer F.SilkS) (width 0.15))
+    (fp_line (start -1.5 0.5) (end -1.5 -0.5) (layer F.SilkS) (width 0.15))
+    (fp_line (start 3.25 -3.25) (end -3.25 -3.25) (layer F.SilkS) (width 0.26))
+    (fp_line (start -3.25 -3.25) (end -3.25 3.25) (layer F.SilkS) (width 0.26))
+    (fp_line (start 3.25 -3.25) (end 3.25 3.25) (layer F.SilkS) (width 0.26))
+    (fp_line (start -3.25 3.25) (end 3.25 3.25) (layer F.SilkS) (width 0.26))
+  )
+  (module pkl_logos:null_Logo_SilkS_6.5mm locked (layer B.Cu)
+    (at 42.4 89)
+    (attr virtual)
+    (fp_text reference REF** (at 0 -4) (layer B.Fab) hide
+      (effects (font (size 1 1) (thickness 0.15)) (justify mirror))
+    )
+    (fp_text value null_Logo_SilkS_6.5mm (at 0 4) (layer B.Fab) hide
+      (effects (font (size 1 1) (thickness 0.15)) (justify mirror))
+    )
+    (fp_arc (start -0.4 -0.2) (end -0.7 -0.2) (angle 180) (layer B.SilkS) (width 0.15))
+    (fp_line (start 1 -0.5) (end 1.5 -0.5) (layer B.SilkS) (width 0.15))
+    (fp_line (start 1 0.5) (end 1 -0.5) (layer B.SilkS) (width 0.15))
+    (fp_line (start 0.2 -0.5) (end 0.7 -0.5) (layer B.SilkS) (width 0.15))
+    (fp_line (start 0.2 0.5) (end 0.2 -0.5) (layer B.SilkS) (width 0.15))
+    (fp_line (start -0.1 -0.2) (end -0.1 0.5) (layer B.SilkS) (width 0.15))
+    (fp_line (start -0.7 0.5) (end -0.7 -0.2) (layer B.SilkS) (width 0.15))
+    (fp_line (start -1 -0.5) (end -1 0.5) (layer B.SilkS) (width 0.15))
+    (fp_line (start -1.5 0.5) (end -1 -0.5) (layer B.SilkS) (width 0.15))
+    (fp_line (start -1.5 -0.5) (end -1.5 0.5) (layer B.SilkS) (width 0.15))
+    (fp_line (start 3.25 3.25) (end -3.25 3.25) (layer B.SilkS) (width 0.26))
+    (fp_line (start -3.25 3.25) (end -3.25 -3.25) (layer B.SilkS) (width 0.26))
+    (fp_line (start 3.25 3.25) (end 3.25 -3.25) (layer B.SilkS) (width 0.26))
+    (fp_line (start -3.25 -3.25) (end 3.25 -3.25) (layer B.SilkS) (width 0.26))
+  )
   (module pkl_connectors:SNES (layer F.Cu)
     (at 55.9 62.000001 270)
@@
     )
   )
-  (module pkl_logos:null_Logo_SilkS_6.5mm locked (layer F.Cu)
-    (at 43.4 89.5)
-    (fp_text reference REF** (at 0 4) (layer F.Fab) hide
-      (effects (font (size 1 1) (thickness 0.15)))
-    )
-    (fp_text value null_Logo_SilkS_6.5mm (at 0 -4) (layer F.Fab) hide
-      (effects (font (size 1 1) (thickness 0.15)))
-    )
-    (fp_line (start -3.25 3.25) (end 3.25 3.25) (layer F.SilkS) (width 0.26))
-    (fp_line (start 3.25 -3.25) (end 3.25 3.25) (layer F.SilkS) (width 0.26))
-    (fp_line (start -3.25 -3.25) (end -3.25 3.25) (layer F.SilkS) (width 0.26))
-    (fp_line (start 3.25 -3.25) (end -3.25 -3.25) (layer F.SilkS) (width 0.26))
-    (fp_line (start -1.5 0.5) (end -1.5 -0.5) (layer F.SilkS) (width 0.15))
-    (fp_line (start -1.5 -0.5) (end -1 0.5) (layer F.SilkS) (width 0.15))
-    (fp_line (start -1 0.5) (end -1 -0.5) (layer F.SilkS) (width 0.15))
-    (fp_line (start -0.7 -0.5) (end -0.7 0.2) (layer F.SilkS) (width 0.15))
-    (fp_line (start -0.1 0.2) (end -0.1 -0.5) (layer F.SilkS) (width 0.15))
-    (fp_line (start 0.2 -0.5) (end 0.2 0.5) (layer F.SilkS) (width 0.15))
-    (fp_line (start 0.2 0.5) (end 0.7 0.5) (layer F.SilkS) (width 0.15))
-    (fp_line (start 1 -0.5) (end 1 0.5) (layer F.SilkS) (width 0.15))
-    (fp_line (start 1 0.5) (end 1.5 0.5) (layer F.SilkS) (width 0.15))
-    (fp_arc (start -0.4 0.2) (end -0.7 0.2) (angle -180) (layer F.SilkS) (width 0.15))
-  )
-  (module pkl_logos:null_Logo_SilkS_6.5mm locked (layer B.Cu)
-    (at 42.4 89)
-    (fp_text reference REF** (at 0 -4) (layer B.Fab) hide
-      (effects (font (size 1 1) (thickness 0.15)) (justify mirror))
-    )
-    (fp_text value null_Logo_SilkS_6.5mm (at 0 4) (layer B.Fab) hide
-      (effects (font (size 1 1) (thickness 0.15)) (justify mirror))
-    )
-    (fp_line (start -3.25 -3.25) (end 3.25 -3.25) (layer B.SilkS) (width 0.26))
-    (fp_line (start 3.25 3.25) (end 3.25 -3.25) (layer B.SilkS) (width 0.26))
-    (fp_line (start -3.25 3.25) (end -3.25 -3.25) (layer B.SilkS) (width 0.26))
-    (fp_line (start 3.25 3.25) (end -3.25 3.25) (layer B.SilkS) (width 0.26))
-    (fp_line (start -1.5 -0.5) (end -1.5 0.5) (layer B.SilkS) (width 0.15))
-    (fp_line (start -1.5 0.5) (end -1 -0.5) (layer B.SilkS) (width 0.15))
-    (fp_line (start -1 -0.5) (end -1 0.5) (layer B.SilkS) (width 0.15))
-    (fp_line (start -0.7 0.5) (end -0.7 -0.2) (layer B.SilkS) (width 0.15))
-    (fp_line (start -0.1 -0.2) (end -0.1 0.5) (layer B.SilkS) (width 0.15))
-    (fp_line (start 0.2 0.5) (end 0.2 -0.5) (layer B.SilkS) (width 0.15))
-    (fp_line (start 0.2 -0.5) (end 0.7 -0.5) (layer B.SilkS) (width 0.15))
-    (fp_line (start 1 0.5) (end 1 -0.5) (layer B.SilkS) (width 0.15))
-    (fp_line (start 1 -0.5) (end 1.5 -0.5) (layer B.SilkS) (width 0.15))
-    (fp_arc (start -0.4 -0.2) (end -0.7 -0.2) (angle 180) (layer B.SilkS) (width 0.15))
-  )
   (module Connector_IDC:IDC-Header_2x06_P2.54mm_Vertical (layer F.Cu)
     (at 41.21 67.65)
@@
     (effects (font (size 1.5 1.5) (thickness 0.375)))
   )
-  (gr_text "iCEBreaker\nSNES Gamepad Pod\nV1.0b\n1Bitsquared 2020\nCC-BY-SA" (at 44.4 61 180) (layer B.SilkS)
+  (gr_text "iCEBreaker\nSNES Gamepad Pod\nV1.1a\n1Bitsquared 2020\nCC-BY-SA" (at 44.4 61 180) (layer B.SilkS)
     (effects (font (size 0.75 0.75) (thickness 0.1875)) (justify mirror))
   )
@@
     (effects (font (size 1 1) (thickness 0.25)))
   )
-  (gr_text "iCEBreaker\nSNES Gamepad Pod\nV1.0b\n1Bitsquared 2020\nCC-BY-SA" (at 43.4 57.5) (layer F.SilkS)
+  (gr_text "iCEBreaker\nSNES Gamepad Pod\nV1.1a\n1Bitsquared 2020\nCC-BY-SA" (at 43.4 57.5) (layer F.SilkS)
     (effects (font (size 0.75 0.75) (thickness 0.1875)))
   )
