File: dvi-16bit/v1.2a/dvi-16bit.sch (KiCad schematic (older format))
At the start: 38 parts, among them J1 PMOD, J10 sj, J2 PMOD, J3 jmp, J4 5V, J5 3v3_5v_sel, J6 HDMI_A_1.4, J7 sj, J8 sj, J9 sj, U1 VREG_3V3, U2 SII164

Commit message: assigned RGB565, moved U2 somewhat and started to re-route
Parts:
- removed J3: jmp, pkl_jumpers:J_NC_0603_30, symbol dvi-16bit-rescue:pkl_jumper_nc-pkl_misc-dvi-12bit-rescue
- removed J4: 5V, Connector_PinHeader_2.54mm:PinHeader_2x01_P2.54mm_Vertical, symbol Connector_Generic:Conn_02x01
- added J4: Conn_02x03_Odd_Even, Connector_PinHeader_2.54mm:PinHeader_2x03_P2.54mm_Horizontal, symbol Connector_Generic:Conn_02x03_Odd_Even
- C11: footprint pkl_dipol:C_0402 -> Capacitor_SMD:C_0603_1608Metric_Pad1.08x0.95mm_HandSolder; symbol dvi-16bit-rescue:pkl_C_Small-pkl_device-dvi-12bit-rescue -> Device:C_Small; Key cap-cer-0402-100n -> (none); Source ANY -> (none)
Connections:
- net labels added: B4, G4, G5, R4
- wire segments 261 -> 260
Changed lines of the file:
@@
 L power:+3V3 #PWR02
 U 1 1 5ADF2EA6
-P 1500 3350
-F 0 "#PWR02" H 1500 3200 50  0001 C CNN
-F 1 "+3V3" H 1515 3526 50  0000 C CNN
-F 2 "" H 1500 3350 50  0001 C CNN
-F 3 "" H 1500 3350 50  0001 C CNN
-	1    1500 3350
+P 1500 3700
+F 0 "#PWR02" H 1500 3550 50  0001 C CNN
+F 1 "+3V3" H 1515 3876 50  0000 C CNN
+F 2 "" H 1500 3700 50  0001 C CNN
+F 3 "" H 1500 3700 50  0001 C CNN
+	1    1500 3700
 	1    0    0    -1
 $EndComp
@@
 	5700 2700 5600 2700
 Text Label 5600 2600 2    50   ~ 0
-G3
+G5
 Wire Wire Line
 	5700 2500 5600 2500
@@
 Wire Wire Line
 	5600 2500 5600 2400
-Connection ~ 5600 2300
-Wire Wire Line
-	5600 2300 5600 2200
 Connection ~ 5600 2400
 Wire Wire Line
@@
 	5700 1900 5600 1900
 Text Label 5600 1800 2    50   ~ 0
-R3
+R4
 Wire Wire Line
 	5700 3000 5600 3000
@@
 Wire Wire Line
 	5600 3300 5600 3200
-Connection ~ 5600 3100
-Wire Wire Line
-	5600 3100 5600 3000
-Connection ~ 5600 3200
-Wire Wire Line
-	5600 3200 5600 3100
 Wire Wire Line
 	5700 3500 5600 3500
@@
 	5700 3700 5600 3700
 Text Label 5600 3400 2    50   ~ 0
-B3
+B4
 Wire Wire Line
 	5700 4100 5600 4100
@@
 Wire Wire Line
 	5600 4100 5600 4000
-Connection ~ 5600 3900
-Wire Wire Line
-	5600 3900 5600 3800
 Connection ~ 5600 4000
 Wire Wire Line
@@
 	1    0    0    -1
 $EndComp
-$Comp
-L dvi-16bit-rescue:pkl_jumper_nc-pkl_misc-dvi-12bit-rescue J3
-U 1 1 5B3C515D
-P 1500 3600
-F 0 "J3" V 1445 3690 60  0000 L CNN
-F 1 "jmp" V 1555 3690 60  0000 L CNN
-F 2 "pkl_jumpers:J_NC_0603_30" V 1610 3690 60  0001 L CNN
-F 3 "" H 1500 3600 60  0000 C CNN
-F 4 "ANY" H 1500 3600 50  0001 C CNN "Source"
-	1    1500 3600
-	0    1    1    0
-$EndComp
 Wire Wire Line
 	2200 3800 1500 3800
@@
 	5300 4100 5300 4200
 Connection ~ 5600 4100
-$Comp
-L Connector_Generic:Conn_02x01 J4
-U 1 1 5B491EFC
-P 1800 2600
-F 0 "J4" H 1850 2820 50  0000 C CNN
-F 1 "5V" H 1850 2727 50  0000 C CNN
-F 2 "Connector_PinHeader_2.54mm:PinHeader_2x01_P2.54mm_Vertical" H 1800 2600 50  0001 C CNN
-F 3 "~" H 1800 2600 50  0001 C CNN
-F 4 "conn-th-01in-2-1-rec" H 1800 2600 50  0001 C CNN "Key"
-F 5 "ANY" H 1800 2600 50  0001 C CNN "Source"
-	1    1800 2600
-	1    0    0    -1
-$EndComp
-Wire Wire Line
-	1600 2600 1500 2600
-Wire Wire Line
-	1500 2600 1500 2800
-Wire Wire Line
-	2100 2600 2200 2600
-Wire Wire Line
-	2200 2600 2200 2500
-$Comp
-L power:+5V #PWR0121
-U 1 1 5B4BB4F9
-P 2200 2500
-F 0 "#PWR0121" H 2200 2350 50  0001 C CNN
-F 1 "+5V" H 2215 2676 50  0000 C CNN
-F 2 "" H 2200 2500 50  0001 C CNN
-F 3 "" H 2200 2500 50  0001 C CNN
-	1    2200 2500
-	1    0    0    -1
-$EndComp
+Wire Wire Line
+	2400 2750 2400 2950
 $Comp
 L power:GND #PWR0122
 U 1 1 5B4BB542
-P 1500 2800
-F 0 "#PWR0122" H 1500 2550 50  0001 C CNN
-F 1 "GND" H 1505 2624 50  0000 C CNN
-F 2 "" H 1500 2800 50  0001 C CNN
-F 3 "" H 1500 2800 50  0001 C CNN
-	1    1500 2800
+P 2400 2950
+F 0 "#PWR0122" H 2400 2700 50  0001 C CNN
+F 1 "GND" H 2405 2774 50  0000 C CNN
+F 2 "" H 2400 2950 50  0001 C CNN
+F 3 "" H 2400 2950 50  0001 C CNN
+	1    2400 2950
 	1    0    0    -1
 $EndComp
@@
 Wire Wire Line
 	1500 3700 1500 3800
-Wire Wire Line
-	1500 3350 1500 3500
 Text Label 7600 3200 0    50   ~ 0
 TFADJ
@@
 	2100 4200 2300 4200
 Text Label 2300 5900 0    50   ~ 0
-B0
+B1
 Text Label 2300 5700 0    50   ~ 0
+B4
+Text Label 1400 5800 2    50   ~ 0
+B2
+Text Label 1400 5700 2    50   ~ 0
 B3
-Text Label 1400 5800 2    50   ~ 0
-B1
-Text Label 1400 5700 2    50   ~ 0
-B2
 Text Label 1400 4400 2    50   ~ 0
-G0
+G2
 Text Label 2300 4400 0    50   ~ 0
-G1
+G3
 Text Label 1400 4300 2    50   ~ 0
-G2
+G4
 Text Label 2300 4300 0    50   ~ 0
-G3
+G5
 Text Label 1400 4200 2    50   ~ 0
-R0
+R1
 Text Label 2300 4200 0    50   ~ 0
-R1
+R2
 Text Label 1400 4100 2    50   ~ 0
-R2
+R3
 Text Label 2300 4100 0    50   ~ 0
-R3
+R4
 Wire Wire Line
 	5600 1800 5700 1800
@@
 	5600 3400 5700 3400
 Text Label 5600 2100 2    50   ~ 0
-R0
+R1
 Text Label 5600 2000 2    50   ~ 0
-R1
+R2
 Text Label 5600 1900 2    50   ~ 0
-R2
+R3
 Text Label 5600 2900 2    50   ~ 0
-G0
+G2
 Text Label 5600 2800 2    50   ~ 0
-G1
+G3
 Text Label 5600 2700 2    50   ~ 0
-G2
+G4
 Text Label 5600 3500 2    50   ~ 0
+B3
+Text Label 5600 3600 2    50   ~ 0
 B2
-Text Label 5600 3600 2    50   ~ 0
-B1
 $Comp
 L dvi-16bit-rescue:pkl_double_jumper_ncno-pkl_misc-dvi-12bit-rescue J5
@@
 Wire Wire Line
 	7700 3900 7700 5200
-$Comp
-L dvi-16bit-rescue:pkl_C_Small-pkl_device-dvi-12bit-rescue C11
-U 1 1 5D249C88
-P 8100 4500
-F 0 "C11" V 8150 4550 50  0000 L CNN
-F 1 "100n" V 8150 4250 50  0000 L CNN
-F 2 "pkl_dipol:C_0402" H 8192 4407 60  0001 L CNN
-F 3 "" H 8100 4500 60  0000 C CNN
-F 4 "cap-cer-0402-100n" H 8100 4500 50  0001 C CNN "Key"
-F 5 "ANY" H 8100 4500 50  0001 C CNN "Source"
-	1    8100 4500
-	1    0    0    -1
-$EndComp
 Wire Wire Line
 	8100 4300 8100 4400
@@
 Connection ~ 4800 4800
 Text Label 5600 3700 2    50   ~ 0
-B0
+B1
 Wire Notes Line
 	4500 2800 2650 2800
@@
 Text Notes 3150 1700 0    50   ~ 0
 DNP\nOptional 3v3 supply
+Text Label 5600 2200 2    50   ~ 0
+R0
+$Comp
+L Connector_Generic:Conn_02x03_Odd_Even J4
+U 1 1 64C0CD5B
+P 1800 2750
+F 0 "J4" H 1850 2975 50  0000 C CNN
+F 1 "Conn_02x03_Odd_Even" H 1850 2976 50  0001 C CNN
+F 2 "Connector_PinHeader_2.54mm:PinHeader_2x03_P2.54mm_Horizontal" H 1800 2750 50  0001 C CNN
+F 3 "~" H 1800 2750 50  0001 C CNN
+	1    1800 2750
+	1    0    0    -1
+$EndComp
+Text Label 2200 2850 0    50   ~ 0
+R0
+Wire Wire Line
+	2100 2850 2200 2850
+$Comp
+L Device:C_Small C11
+U 1 1 5D249C88
+P 8100 4500
+F 0 "C11" V 8150 4550 50  0000 L CNN
+F 1 "100n" V 8150 4250 50  0000 L CNN
+F 2 "Capacitor_SMD:C_0603_1608Metric_Pad1.08x0.95mm_HandSolder" H 8192 4407 60  0001 L CNN
+F 3 "" H 8100 4500 60  0001 C CNN
+F 4 "" H 8100 4500 50  0001 C CNN "Key"
+F 5 "" H 8100 4500 50  0001 C CNN "Source"
+	1    8100 4500
+	1    0    0    -1
+$EndComp
+Text Label 5600 3000 2    50   ~ 0
+G1
+Text Label 5600 3100 2    50   ~ 0
+G0
+Text Label 1500 2850 2    50   ~ 0
+G1
+Wire Wire Line
+	1500 2850 1600 2850
+Text Label 1500 2750 2    50   ~ 0
+G0
+Wire Wire Line
+	1500 2750 1600 2750
+Wire Wire Line
+	2100 2750 2400 2750
+Text Label 5600 3800 2    50   ~ 0
+B0
+Text Label 1500 2650 2    50   ~ 0
+B0
+Wire Wire Line
+	2100 2650 2400 2650
+Wire Wire Line
+	2400 2650 2400 2750
+Connection ~ 2400 2750
+Wire Wire Line
+	1500 2650 1600 2650
 $EndSCHEMATC

Commit message: more routing and silkscreen fixes
Parts:
- C1: footprint pkl_dipol:C_0603 -> Capacitor_SMD:C_1206_3216Metric_Pad1.33x1.80mm_HandSolder; symbol dvi-16bit-rescue:pkl_C-pkl_device-dvi-12bit-rescue -> Device:C; Key cap-cer-0603-10u -> (none); Source ANY -> (none)
Other:
- moved on the sheet: C1
Changed lines of the file:
@@
 $EndComp
 $Comp
-L dvi-16bit-rescue:pkl_C-pkl_device-dvi-12bit-rescue C1
+L Device:C C1
 U 1 1 5ADF32E3
-P 1850 5000
-F 0 "C1" H 1965 5047 50  0000 L CNN
-F 1 "10u" H 1965 4954 50  0000 L CNN
-F 2 "pkl_dipol:C_0603" H 1965 4907 30  0001 L CNN
-F 3 "" H 1850 5000 60  0000 C CNN
-F 4 "cap-cer-0603-10u" H 1850 5000 50  0001 C CNN "Key"
-F 5 "ANY" H 1850 5000 50  0001 C CNN "Source"
-	1    1850 5000
+P 1850 5050
+F 0 "C1" H 1965 5097 50  0000 L CNN
+F 1 "10u" H 1965 5004 50  0000 L CNN
+F 2 "Capacitor_SMD:C_1206_3216Metric_Pad1.33x1.80mm_HandSolder" H 1965 4957 30  0001 L CNN
+F 3 "" H 1850 5050 60  0001 C CNN
+F 4 "" H 1850 5050 50  0001 C CNN "Key"
+F 5 "" H 1850 5050 50  0001 C CNN "Source"
+	1    1850 5050
 	1    0    0    -1
 $EndComp
@@
 L power:GND #PWR04
 U 1 1 5ADF354C
-P 1850 5100
-F 0 "#PWR04" H 1850 4850 50  0001 C CNN
-F 1 "GND" H 1855 4924 50  0000 C CNN
-F 2 "" H 1850 5100 50  0001 C CNN
-F 3 "" H 1850 5100 50  0001 C CNN
-	1    1850 5100
+P 1850 5200
+F 0 "#PWR04" H 1850 4950 50  0001 C CNN
+F 1 "GND" H 1855 5024 50  0000 C CNN
+F 2 "" H 1850 5200 50  0001 C CNN
+F 3 "" H 1850 5200 50  0001 C CNN
+	1    1850 5200
 	1    0    0    -1
 $EndComp

Commit message: more routing and placing
Parts:
- removed J10: sj, pkl_jumpers:J_0603, symbol dvi-16bit-rescue:pkl_jumper-pkl_misc-dvi-12bit-rescue
- added J10: Jumper_NO_Small, Connector_PinHeader_2.00mm:PinHeader_1x02_P2.00mm_Vertical, symbol Device:Jumper_NO_Small
- C10, C6: footprint pkl_dipol:C_0402 -> Capacitor_SMD:C_0603_1608Metric_Pad1.08x0.95mm_HandSolder; symbol dvi-16bit-rescue:pkl_C_Small-pkl_device-dvi-12bit-rescue -> Device:C_Small; Key cap-cer-0402-100n -> (none); Source ANY -> (none)
- R3: footprint pkl_dipol:R_0402 -> Resistor_SMD:R_0603_1608Metric_Pad0.98x0.95mm_HandSolder; symbol dvi-16bit-rescue:pkl_R_Small-pkl_device-dvi-12bit-rescue -> Device:R_Small; Key res-0402-10k -> (none); Source ANY -> (none)
Other:
- moved on the sheet: J4
Changed lines of the file:
@@
 $EndComp
 $Comp
-L dvi-16bit-rescue:pkl_C_Small-pkl_device-dvi-12bit-rescue C6
+L Device:C_Small C6
 U 1 1 5AFD5EBB
 P 8100 3600
 F 0 "C6" V 8150 3650 50  0000 L CNN
 F 1 "100n" V 8150 3350 50  0000 L CNN
-F 2 "pkl_dipol:C_0402" H 8192 3507 60  0001 L CNN
-F 3 "" H 8100 3600 60  0000 C CNN
-F 4 "cap-cer-0402-100n" H 8100 3600 50  0001 C CNN "Key"
-F 5 "ANY" H 8100 3600 50  0001 C CNN "Source"
+F 2 "Capacitor_SMD:C_0603_1608Metric_Pad1.08x0.95mm_HandSolder" H 8192 3507 60  0001 L CNN
+F 3 "" H 8100 3600 60  0001 C CNN
+F 4 "" H 8100 3600 50  0001 C CNN "Key"
+F 5 "" H 8100 3600 50  0001 C CNN "Source"
 	1    8100 3600
 	1    0    0    -1
@@
 $EndComp
 $Comp
-L dvi-16bit-rescue:pkl_C_Small-pkl_device-dvi-12bit-rescue C10
+L Device:C_Small C10
 U 1 1 5AFDA5D4
 P 8300 5400
 F 0 "C10" V 8350 5450 50  0000 L CNN
 F 1 "100n" V 8350 5150 50  0000 L CNN
-F 2 "pkl_dipol:C_0402" H 8392 5307 60  0001 L CNN
-F 3 "" H 8300 5400 60  0000 C CNN
-F 4 "cap-cer-0402-100n" H 8300 5400 50  0001 C CNN "Key"
-F 5 "ANY" H 8300 5400 50  0001 C CNN "Source"
+F 2 "Capacitor_SMD:C_0603_1608Metric_Pad1.08x0.95mm_HandSolder" H 8392 5307 60  0001 L CNN
+F 3 "" H 8300 5400 60  0001 C CNN
+F 4 "" H 8300 5400 50  0001 C CNN "Key"
+F 5 "" H 8300 5400 50  0001 C CNN "Source"
 	1    8300 5400
 	1    0    0    -1
@@
 	4800 4800 5700 4800
 $Comp
-L dvi-16bit-rescue:pkl_R_Small-pkl_device-dvi-12bit-rescue R3
+L Device:R_Small R3
 U 1 1 5B2C7F22
 P 4800 4400
 F 0 "R3" V 4800 4350 50  0000 L CNN
 F 1 "10k" V 4850 4500 50  0000 L CNN
-F 2 "pkl_dipol:R_0402" H 4859 4307 60  0001 L CNN
-F 3 "" H 4800 4400 60  0000 C CNN
-F 4 "res-0402-10k" H 4800 4400 50  0001 C CNN "Key"
-F 5 "ANY" H 4800 4400 50  0001 C CNN "Source"
+F 2 "Resistor_SMD:R_0603_1608Metric_Pad0.98x0.95mm_HandSolder" H 4859 4307 60  0001 L CNN
+F 3 "" H 4800 4400 60  0001 C CNN
+F 4 "" H 4800 4400 50  0001 C CNN "Key"
+F 5 "" H 4800 4400 50  0001 C CNN "Source"
 	1    4800 4400
 	1    0    0    -1
@@
 Connection ~ 5600 4100
 Wire Wire Line
-	2400 2750 2400 2950
+	2400 3050 2400 3250
 $Comp
 L power:GND #PWR0122
 U 1 1 5B4BB542
-P 2400 2950
-F 0 "#PWR0122" H 2400 2700 50  0001 C CNN
-F 1 "GND" H 2405 2774 50  0000 C CNN
-F 2 "" H 2400 2950 50  0001 C CNN
-F 3 "" H 2400 2950 50  0001 C CNN
-	1    2400 2950
+P 2400 3250
+F 0 "#PWR0122" H 2400 3000 50  0001 C CNN
+F 1 "GND" H 2405 3074 50  0000 C CNN
+F 2 "" H 2400 3250 50  0001 C CNN
+F 3 "" H 2400 3250 50  0001 C CNN
+	1    2400 3250
 	1    0    0    -1
 $EndComp
@@
 Text Label 5600 5500 2    50   ~ 0
 DK1
-$Comp
-L dvi-16bit-rescue:pkl_jumper-pkl_misc-dvi-12bit-rescue J10
-U 1 1 5D74A0AB
-P 4400 6000
-F 0 "J10" H 4350 6050 50  0000 R CNN
-F 1 "sj" H 4500 6050 50  0000 L CNN
-F 2 "pkl_jumpers:J_0603" H 4400 6000 60  0001 C CNN
-F 3 "" H 4400 6000 60  0000 C CNN
-	1    4400 6000
-	0    1    1    0
-$EndComp
 Wire Wire Line
 	4400 6100 4400 6300
@@
 L Connector_Generic:Conn_02x03_Odd_Even J4
 U 1 1 64C0CD5B
-P 1800 2750
-F 0 "J4" H 1850 2975 50  0000 C CNN
-F 1 "Conn_02x03_Odd_Even" H 1850 2976 50  0001 C CNN
-F 2 "Connector_PinHeader_2.54mm:PinHeader_2x03_P2.54mm_Horizontal" H 1800 2750 50  0001 C CNN
-F 3 "~" H 1800 2750 50  0001 C CNN
-	1    1800 2750
-	1    0    0    -1
-$EndComp
-Text Label 2200 2850 0    50   ~ 0
+P 1800 3050
+F 0 "J4" H 1850 3275 50  0000 C CNN
+F 1 "Conn_02x03_Odd_Even" H 1850 3276 50  0001 C CNN
+F 2 "Connector_PinHeader_2.54mm:PinHeader_2x03_P2.54mm_Horizontal" H 1800 3050 50  0001 C CNN
+F 3 "~" H 1800 3050 50  0001 C CNN
+	1    1800 3050
+	1    0    0    -1
+$EndComp
+Text Label 2200 3150 0    50   ~ 0
 R0
 Wire Wire Line
-	2100 2850 2200 2850
+	2100 3150 2200 3150
 $Comp
 L Device:C_Small C11
@@
 Text Label 5600 3100 2    50   ~ 0
 G0
-Text Label 1500 2850 2    50   ~ 0
+Text Label 1500 3150 2    50   ~ 0
 G1
 Wire Wire Line
-	1500 2850 1600 2850
-Text Label 1500 2750 2    50   ~ 0
+	1500 3150 1600 3150
+Text Label 1500 3050 2    50   ~ 0
 G0
 Wire Wire Line
-	1500 2750 1600 2750
-Wire Wire Line
-	2100 2750 2400 2750
+	1500 3050 1600 3050
+Wire Wire Line
+	2100 3050 2400 3050
 Text Label 5600 3800 2    50   ~ 0
 B0
-Text Label 1500 2650 2    50   ~ 0
+Text Label 1500 2950 2    50   ~ 0
 B0
 Wire Wire Line
-	2100 2650 2400 2650
-Wire Wire Line
-	2400 2650 2400 2750
-Connection ~ 2400 2750
-Wire Wire Line
-	1500 2650 1600 2650
+	2100 2950 2400 2950
+Wire Wire Line
+	2400 2950 2400 3050
+Connection ~ 2400 3050
+Wire Wire Line
+	1500 2950 1600 2950
+$Comp
+L Device:Jumper_NO_Small J10
+U 1 1 651B16C4
+P 4400 6000
+F 0 "J10" H 4200 6050 50  0000 L CNN
+F 1 "Jumper_NO_Small" V 4445 6048 50  0001 L CNN
+F 2 "Connector_PinHeader_2.00mm:PinHeader_1x02_P2.00mm_Vertical" H 4400 6000 50  0001 C CNN
+F 3 "~" H 4400 6000 50  0001 C CNN
+	1    4400 6000
+	0    1    1    0
+$EndComp
 $EndSCHEMATC

Commit message: more routing and placing
Parts:
- C15: footprint pkl_dipol:C_0603 -> Capacitor_SMD:C_0805_2012Metric_Pad1.18x1.45mm_HandSolder; symbol dvi-16bit-rescue:pkl_C-pkl_device-dvi-12bit-rescue -> Device:C_Small; Key cap-cer-0603-10u -> (none); Source ANY -> (none)
- C7, C9: footprint pkl_dipol:C_0402 -> Capacitor_SMD:C_0603_1608Metric_Pad1.08x0.95mm_HandSolder; symbol dvi-16bit-rescue:pkl_C_Small-pkl_device-dvi-12bit-rescue -> Device:C_Small; Key cap-cer-0402-100n -> (none); Source ANY -> (none)
- L2: footprint pkl_dipol:L_0402 -> Inductor_SMD:L_0603_1608Metric_Pad1.05x0.95mm_HandSolder; symbol dvi-16bit-rescue:pkl_L_Small-pkl_device-dvi-12bit-rescue -> Device:L_Small; Key ferrite-0402-600 -> (none); Source ANY -> (none)
- R9: footprint pkl_dipol:R_0402 -> Resistor_SMD:R_0603_1608Metric_Pad0.98x0.95mm_HandSolder; symbol dvi-16bit-rescue:pkl_R_Small-pkl_device-dvi-12bit-rescue -> Device:R_Small; Key res-0402-510 -> (none); Source ANY -> (none)
Connections:
- net +3V3: now also L2.2; no longer L2.1
- net +5V: now also J4.3 (Pin_3)
- net G0: now also J4.2 (Pin_2); no longer J4.3 (Pin_3)
- net GND: no longer J4.2 (Pin_2)
- net PVCC: now also L2.1; no longer L2.2
Changed lines of the file:
@@
 	7600 3200 7600 2300
 $Comp
-L dvi-16bit-rescue:pkl_R_Small-pkl_device-dvi-12bit-rescue R9
+L Device:R_Small R9
 U 1 1 5B0DC406
 P 7600 2200
 F 0 "R9" H 7659 2247 50  0000 L CNN
 F 1 "510E" H 7659 2154 50  0000 L CNN
-F 2 "pkl_dipol:R_0402" H 7659 2107 60  0001 L CNN
-F 3 "" H 7600 2200 60  0000 C CNN
-F 4 "res-0402-510" H 7600 2200 50  0001 C CNN "Key"
-F 5 "ANY" H 7600 2200 50  0001 C CNN "Source"
+F 2 "Resistor_SMD:R_0603_1608Metric_Pad0.98x0.95mm_HandSolder" H 7659 2107 60  0001 L CNN
+F 3 "" H 7600 2200 60  0001 C CNN
+F 4 "" H 7600 2200 50  0001 C CNN "Key"
+F 5 "" H 7600 2200 50  0001 C CNN "Source"
 	1    7600 2200
 	1    0    0    -1
@@
 	8900 3400 8900 3300
 $Comp
-L dvi-16bit-rescue:pkl_C_Small-pkl_device-dvi-12bit-rescue C9
+L Device:C_Small C9
 U 1 1 5B1E6CEE
 P 8300 4500
 F 0 "C9" V 8350 4550 50  0000 L CNN
 F 1 "100n" V 8350 4250 50  0000 L CNN
-F 2 "pkl_dipol:C_0402" H 8392 4407 60  0001 L CNN
-F 3 "" H 8300 4500 60  0000 C CNN
-F 4 "cap-cer-0402-100n" H 8300 4500 50  0001 C CNN "Key"
-F 5 "ANY" H 8300 4500 50  0001 C CNN "Source"
+F 2 "Capacitor_SMD:C_0603_1608Metric_Pad1.08x0.95mm_HandSolder" H 8392 4407 60  0001 L CNN
+F 3 "" H 8300 4500 60  0001 C CNN
+F 4 "" H 8300 4500 50  0001 C CNN "Key"
+F 5 "" H 8300 4500 50  0001 C CNN "Source"
 	1    8300 4500
 	1    0    0    -1
 $EndComp
 $Comp
-L dvi-16bit-rescue:pkl_C-pkl_device-dvi-12bit-rescue C15
+L Device:C_Small C15
 U 1 1 5B1E6D2A
 P 8500 4500
 F 0 "C15" V 8550 4550 50  0000 L CNN
 F 1 "10u" V 8550 4250 50  0000 L CNN
-F 2 "pkl_dipol:C_0603" H 8592 4407 60  0001 L CNN
-F 3 "" H 8500 4500 60  0000 C CNN
-F 4 "cap-cer-0603-10u" H 8500 4500 50  0001 C CNN "Key"
-F 5 "ANY" H 8500 4500 50  0001 C CNN "Source"
+F 2 "Capacitor_SMD:C_0805_2012Metric_Pad1.18x1.45mm_HandSolder" H 8592 4407 60  0001 L CNN
+F 3 "" H 8500 4500 60  0001 C CNN
+F 4 "" H 8500 4500 50  0001 C CNN "Key"
+F 5 "" H 8500 4500 50  0001 C CNN "Source"
 	1    8500 4500
 	1    0    0    -1
@@
 Connection ~ 8300 4300
 $Comp
-L dvi-16bit-rescue:pkl_L_Small-pkl_device-dvi-12bit-rescue L2
+L Device:L_Small L2
 U 1 1 5B2038E0
 P 8700 4300
 F 0 "L2" V 8890 4300 50  0000 C CNN
 F 1 "600" V 8797 4300 50  0000 C CNN
-F 2 "pkl_dipol:L_0402" H 8749 4207 60  0001 L CNN
-F 3 "" V 8700 4300 60  0000 C CNN
-F 4 "ferrite-0402-600" H 8700 4300 50  0001 C CNN "Key"
-F 5 "ANY" H 8700 4300 50  0001 C CNN "Source"
+F 2 "Inductor_SMD:L_0603_1608Metric_Pad1.05x0.95mm_HandSolder" H 8749 4207 60  0001 L CNN
+F 3 "" V 8700 4300 60  0001 C CNN
+F 4 "" H 8700 4300 50  0001 C CNN "Key"
+F 5 "" H 8700 4300 50  0001 C CNN "Source"
 	1    8700 4300
 	0    -1   -1   0
@@
 TFADJ
 $Comp
-L dvi-16bit-rescue:pkl_C_Small-pkl_device-dvi-12bit-rescue C7
+L Device:C_Small C7
 U 1 1 5AFDA5AA
 P 8100 5400
 F 0 "C7" V 8150 5450 50  0000 L CNN
 F 1 "100n" V 8150 5150 50  0000 L CNN
-F 2 "pkl_dipol:C_0402" H 8192 5307 60  0001 L CNN
-F 3 "" H 8100 5400 60  0000 C CNN
-F 4 "cap-cer-0402-100n" H 8100 5400 50  0001 C CNN "Key"
-F 5 "ANY" H 8100 5400 50  0001 C CNN "Source"
+F 2 "Capacitor_SMD:C_0603_1608Metric_Pad1.08x0.95mm_HandSolder" H 8192 5307 60  0001 L CNN
+F 3 "" H 8100 5400 60  0001 C CNN
+F 4 "" H 8100 5400 50  0001 C CNN "Key"
+F 5 "" H 8100 5400 50  0001 C CNN "Source"
 	1    8100 5400
 	1    0    0    -1
@@
 Wire Wire Line
 	1500 3150 1600 3150
-Text Label 1500 3050 2    50   ~ 0
+Text Label 2200 2950 0    50   ~ 0
 G0
-Wire Wire Line
-	1500 3050 1600 3050
 Wire Wire Line
 	2100 3050 2400 3050
@@
 Text Label 1500 2950 2    50   ~ 0
 B0
-Wire Wire Line
-	2100 2950 2400 2950
-Wire Wire Line
-	2400 2950 2400 3050
-Connection ~ 2400 3050
 Wire Wire Line
 	1500 2950 1600 2950
@@
 	0    1    1    0
 $EndComp
+Wire Wire Line
+	1100 3050 1100 2950
+Wire Wire Line
+	1100 3050 1600 3050
+$Comp
+L power:+5V #PWR?
+U 1 1 64CDB0FD
+P 1100 2950
+F 0 "#PWR?" H 1100 2800 50  0001 C CNN
+F 1 "+5V" H 1115 3126 50  0000 C CNN
+F 2 "" H 1100 2950 50  0001 C CNN
+F 3 "" H 1100 2950 50  0001 C CNN
+	1    1100 2950
+	1    0    0    -1
+$EndComp
+Wire Wire Line
+	2100 2950 2200 2950
 $EndSCHEMATC

Commit message: more routing and fixes
Connections:
- net G1: now also J4.6 (Pin_6); no longer J4.5 (Pin_5)
- net R0: now also J4.5 (Pin_5); no longer J4.6 (Pin_6)
Changed lines of the file:
@@
 	1    0    0    -1
 $EndComp
-Text Label 2200 3150 0    50   ~ 0
+Text Label 1500 3150 2    50   ~ 0
 R0
 Wire Wire Line
@@
 Text Label 5600 3100 2    50   ~ 0
 G0
-Text Label 1500 3150 2    50   ~ 0
+Text Label 2200 3150 0    50   ~ 0
 G1
 Wire Wire Line

Commit message: more routing and fixes
Parts:
- removed C2, C4: 4u7, pkl_dipol:C_0603, symbol dvi-16bit-rescue:pkl_C-pkl_device-dvi-12bit-rescue
- removed C3: 470p, pkl_dipol:C_0402, symbol dvi-16bit-rescue:pkl_C_Small-pkl_device-dvi-12bit-rescue
- removed R1, R2, R4, R8: 10k, pkl_dipol:R_0402, symbol dvi-16bit-rescue:pkl_R_Small-pkl_device-dvi-12bit-rescue
- removed U1: VREG_3V3, pkl_housings_sot:SOT-23-5, symbol dvi-16bit-rescue:pkl_VREG_5PIN_FIXED-pkl_device-dvi-12bit-rescue
- added RN1: R_Pack04, dvi-16bit:RESCAF80P320X160X60-8N, symbol Device:R_Pack04
- C10: renamed from C14; footprint pkl_dipol:C_0603 -> Capacitor_SMD:C_0805_2012Metric_Pad1.18x1.45mm_HandSolder; symbol dvi-16bit-rescue:pkl_C-pkl_device-dvi-12bit-rescue -> Device:C; Key cap-cer-0603-10u -> (none); Source ANY -> (none)
- C11: renamed from C15; symbol Device:C_Small -> Device:C
- C2: renamed from C5; footprint pkl_dipol:C_0402 -> Capacitor_SMD:C_0603_1608Metric_Pad1.08x0.95mm_HandSolder; symbol dvi-16bit-rescue:pkl_C_Small-pkl_device-dvi-12bit-rescue -> Device:C_Small; Key cap-cer-0402-100n -> (none); Source ANY -> (none)
- C4: renamed from C8; footprint pkl_dipol:C_0402 -> Capacitor_SMD:C_0603_1608Metric_Pad1.08x0.95mm_HandSolder; symbol dvi-16bit-rescue:pkl_C_Small-pkl_device-dvi-12bit-rescue -> Device:C_Small; Key cap-cer-0402-100n -> (none); Source ANY -> (none)
- C9: renamed from C16; footprint pkl_dipol:C_0603 -> Capacitor_SMD:C_0805_2012Metric; symbol dvi-16bit-rescue:pkl_C-pkl_device-dvi-12bit-rescue -> Device:C; Key cap-cer-0603-10u -> (none); Source ANY -> (none)
- L1: footprint pkl_dipol:L_0402 -> L_0603_1608Metric_Pad1.05x0.95mm_HandSolder; symbol dvi-16bit-rescue:pkl_L_Small-pkl_device-dvi-12bit-rescue -> Device:L_Small; Key ferrite-0402-600 -> (none); Source ANY -> (none)
- L3: footprint pkl_dipol:L_0402 -> Inductor_SMD:L_0603_1608Metric_Pad1.05x0.95mm_HandSolder; symbol dvi-16bit-rescue:pkl_L_Small-pkl_device-dvi-12bit-rescue -> Device:L_Small; Key ferrite-0402-600 -> (none); Source ANY -> (none)
- R5: footprint pkl_dipol:R_0402 -> Resistor_SMD:R_0603_1608Metric_Pad0.98x0.95mm_HandSolder; symbol dvi-16bit-rescue:pkl_R_Small-pkl_device-dvi-12bit-rescue -> Device:R_Small; Key res-0402-33k -> (none); Source ANY -> (none)
- R6: footprint pkl_dipol:R_0402 -> Resistor_SMD:R_0603_1608Metric_Pad0.98x0.95mm_HandSolder; symbol dvi-16bit-rescue:pkl_R_Small-pkl_device-dvi-12bit-rescue -> Device:R_Small; Key dnp -> (none); Source ANY -> (none)
- R7: footprint pkl_dipol:R_0402 -> Resistor_SMD:R_0603_1608Metric_Pad0.98x0.95mm_HandSolder; symbol dvi-16bit-rescue:pkl_R_Small-pkl_device-dvi-12bit-rescue -> Device:R_Small; Key res-0402-10k -> (none); Source ANY -> (none)
- renumbered C6 to C3, C11 to C5, C9 to C6, C10 to C8, R3 to R1
Connections:
- net +3V3: now also L1.2, L3.2, RN1.6 (R3.2), RN1.7 (R2.2), RN1.8 (R1.2); no longer C1.1, L1.1, L3.1
- net +5V: now also C1.1
- net BSEL-SCL: now also RN1.3 (R3.1)
- net DSEL-SDA: now also RN1.4 (R4.1)
- net EDGE-HTPLG: now also RN1.1 (R1.1)
- net GND: now also RN1.5 (R4.2)
- net TVDD: now also L3.1; no longer L3.2
- net VCC: now also L1.1; no longer L1.2
- net ~PD: now also RN1.2 (R2.1)
Other:
- note removed: "DNP\nOptional 3v3 supply"
- moved on the sheet: C1, C10, C11, C9, R1, R5, R6, R7
